File: filters.kicad_sch (KiCad schematic)
At the start: 28 parts, among them J100 Conn_01x02, J101 Conn_01x02, J102 Conn_01x02, J103 Conn_02x04_Odd_Even, J92 Conn_02x04_Odd_Even, J93 Conn_01x02, J94 Conn_01x02, J95 Conn_01x02, J96 Conn_01x02, J97 Conn_02x04_Odd_Even, J98 Conn_02x04_Odd_Even, J99 Conn_01x02

Commit message: WIP v0.2.0 changes
Parts:
- removed J103, J92, J97, J98: Conn_02x04_Odd_Even, HL_Connector_Pad_2.54mm:Pad_2x04_P2.54_1.7x1.7_Rect-Oct, symbol Connector_Generic:Conn_02x04_Odd_Even
- added J86, J91, J98, J99: Conn_01x05, HL_Connector_Pad_2.54mm:Pad_1x05_P2.54_1.7x1.7_Rect-Oct, symbol Connector_Generic:Conn_01x05
- RV19, RV20, RV21, RV22, RV23, RV24, RV25, RV26: LCSC (none) -> C118963; THT_LCSC C118963 -> (none)
- renumbered J93 to J81, J94 to J82, J95 to J83, J96 to J84, J99 to J87, J100 to J88, J101 to J89, J102 to J90
Connections:
- net GND: now also J86.1 (Pin_1), J91.1 (Pin_1), J98.1 (Pin_1), J99.1 (Pin_1)
- net HPIN1: now also J86.2 (Pin_2)
- net HPIN2: now also J86.3 (Pin_3)
- net HPIN3: now also J86.4 (Pin_4)
- net HPIN4: now also J86.5 (Pin_5)
- net HPOUT1: now also J91.2 (Pin_2)
- net HPOUT2: now also J91.3 (Pin_3)
- net HPOUT3: now also J91.4 (Pin_4)
- net HPOUT4: now also J91.5 (Pin_5)
- net LPIN1: now also J99.2 (Pin_2)
- net LPIN2: now also J99.3 (Pin_3)
- net LPIN3: now also J99.4 (Pin_4)
- net LPIN4: now also J99.5 (Pin_5)
- net LPOUT1: now also J98.2 (Pin_2)
- net LPOUT2: now also J98.3 (Pin_3)
- net LPOUT3: now also J98.4 (Pin_4)
- net LPOUT4: now also J98.5 (Pin_5)
