File: curlim_12V.kicad_sch (KiCad schematic)
At the start: 17 parts, among them J19 Conn_01x02, J20 Conn_02x03_Odd_Even, Q2 AO3401A, Q3 2N7002, Q4 AO3401A, U12 INA199A1DCKR, U13 LMV321-TR, U14 74HC02

Commit message: WIP v0.2.0 changes
Parts:
- removed R34: 10k, Resistor_SMD:R_0603_1608Metric_Pad0.98x0.95mm_HandSolder, symbol Device:R
- added J22: Conn_01x02, HL_Connector_Pad_2.54mm:Pad_1x02_P2.54_1.7x1.7_Rect, symbol Connector_Generic:Conn_01x02
- added R73: 10k, Resistor_SMD:R_0603_1608Metric_Pad0.98x0.95mm_HandSolder, symbol Device:R_Small
- J18: renamed from J19; footprint HL_Connector_Pad_2.00mm:Pad_1x02_P2.00_1.35x1.35_Rnd-Oct -> HL_Connector_Pad_2.00mm:Pad_1x02_P2.00_1.35x1.35_Rect-Oct
- J19: renamed from J20; value Conn_02x03_Odd_Even -> Conn_01x03_Odd_Even; footprint HL_Connector_Pad_2.54mm:Pad_2x03_P2.54_1.7x1.7_Rect-1Oct-2Rnd -> HL_Connector_Pad_2.54mm:Pad_1x03_P2.54_1.7x1.7_Rnd-Rnd-Oct; symbol Connector_Generic:Conn_02x03_Odd_Even -> Connector_Generic:Conn_01x03
- RV5: LCSC (none) -> C118963; THT_LCSC C118963 -> (none)
Connections:
- net +3.3V: now also RV5.1; no longer J18.1 (Pin_1), RV5.2
- net CV-: now also RV5.2; no longer RV5.3
- net EN: now also R73.1
- net GND: now also J18.1 (Pin_1), RV5.3, J22.1 (Pin_1), J22.2 (Pin_2), R73.2; no longer J19.1 (Pin_1), J19.3 (Pin_3), J19.5 (Pin_5)
- net V_{Iin}: now also J19.3 (Pin_3); no longer J19.2 (Pin_2)
- net Vout: now also J19.1 (Pin_1), J19.2 (Pin_2); no longer J19.4 (Pin_4), J19.6 (Pin_6)
- no-connect marks 1 -> 0
Other:
- note added: "INA199A1 amplification is 50x"
- moved on the sheet: J18, RV5

Commit message: Assign part numbers and finish other 0.2.0 changes
Parts:
- J20: renamed from J19; LCSC (none) -> C2937625
- J21: renamed from J22; LCSC (none) -> C492401
- renumbered C35 to C40, C36 to C41, C37 to C42, J18 to J19, R31 to R38, R32 to R39, R33 to R40, R73 to R41

Commit message: Update the title blocks
Other:
- company: (none) -> Hat Labs Oy
- title: (none) -> HALSPA - Hat Labs Spaghetti Board
Changed lines of the file:
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@@
 	(generator_version "9.0")
 	(paper "A4")
+	(title_block
+		(title "HALSPA - Hat Labs Spaghetti Board")
+		(date "2025-04-17")
+		(rev "v0.2.0")
+		(company "Hat Labs Oy")
+		(comment 1 "See the accompanying LICENSE.md file for license details.")
+	)
 	(rectangle
 		(start 85.09 15.24)

Commit message: Add JLCPCB corrections
Parts:
- J20: JLCPCB_CORRECTION (none) -> 0;2.54;270
- J21: JLCPCB_CORRECTION (none) -> 0;1.27;270
- RV5: now in the parts list
Changed lines of the file:
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@@
 		(unit 1)
 		(exclude_from_sim no)
-		(in_bom no)
+		(in_bom yes)
 		(on_board yes)
 		(dnp no)
@@
 		)
 		(property "LCSC" "C492401"
+			(at 205.74 46.99 0)
+			(effects
+				(font
+					(size 1.27 1.27)
+				)
+				(hide yes)
+			)
+		)
+		(property "JLCPCB_CORRECTION" "0;1.27;270"
 			(at 205.74 46.99 0)
 			(effects
@@
 			(at 205.74 36.83 0)
 			(effects
+				(font
+					(size 1.27 1.27)
+				)
+				(hide yes)
+			)
+		)
+		(property "JLCPCB_CORRECTION" "0;2.54;270"
+			(at 205.74 36.83 0)
+			(effects

Commit message: Improve MCU2 layout; document curlim12v CSA
Parts:
- added C67: 1uF, Capacitor_SMD:C_0603_1608Metric_Pad1.08x0.95mm_HandSolder, symbol Device:C_Small
- added R189: 10k, Resistor_SMD:R_0603_1608Metric_Pad0.98x0.95mm_HandSolder, symbol Device:R_Small
Connections:
- net FAULT: now also R189.1; no longer U14.2
- net GND: now also C67.2
- new net FAULT_F: C67.1, R189.2, U14.2
Other:
- note added: "INA199A1 amplification is 50x. Adjust V_{CV-} to 0.5 V/A * Imax."
- note removed: "INA199A1 amplification is 50x"
