File: dut_power.kicad_sch (KiCad schematic)
At the start: 51 parts, among them J10 Conn_01x04, J6 Conn_02x04_Odd_Even, J7 Conn_01x02, J8 Conn_02x04_Odd_Even, J9 Conn_02x04_Odd_Even, Q1 AO3401A, U1 TCA9535PWR(UMW)

Commit message: WIP v0.2.0 changes
Parts:
- removed J10: Conn_01x04, HL_Connector_Pad_2.54mm:Pad_1x04_P2.54_1.7x1.7_Rect-Oct, symbol Connector_Generic:Conn_01x04
- J7: footprint Connector_Phoenix_MC:PhoenixContact_MCV_1,5_2-G-3.81_1x02_P3.81mm_Vertical -> Connector_Phoenix_MC:PhoenixContact_MC_1,5_2-G-3.81_1x02_P3.81mm_Horizontal; JLCPCB_CORRECTION 1.905;0;180 -> (none); LCSC (none) -> C8387; THT_LCSC C8396 -> (none)

Commit message: Assign part numbers and finish other 0.2.0 changes
Parts:
- added C4, C5, C6, C8, C9: 10uF/50V, Capacitor_SMD:C_1206_3216Metric, symbol Device:C
- added D3: SMF13CA, Diode_SMD:D_SOD-123, symbol Device:D_TVS
- added L1: FXL0420-1R5-M, Hatlabs:L_MWSA0402, symbol Device:L
- added R19: 0.1R, Resistor_SMD:R_1206_3216Metric, symbol Device:R
- added TP1: TestPoint, TestPoint:TestPoint_Pad_D1.0mm, symbol Connector:TestPoint
- J10: renamed from J9; LCSC (none) -> C7501275
- J7: renamed from J6; LCSC (none) -> C7501275
- J9: renamed from J8; LCSC (none) -> C7501275
- renumbered C4 to C10, C5 to C11, C6 to C7, D9 to D10, D10 to D11, D11 to D12, D12 to D13, D13 to D14, D14 to D15, D15 to D16, D16 to D17, D17 to D18, D18 to D19, D19 to D20, D3 to D4, D4 to D5, D5 to D6, D6 to D7, D7 to D8, D8 to D9, J7 to J8, R19 to R20, R20 to R21
Connections:
- net +12V: now also C8.1, C9.1, L1.2; no longer DZ1.1 (K), Q1.2 (S), R1.1
- net GND: now also C4.2, C5.2, C6.2, D3.1 (A1), R19.2
- net Vin: now also D3.2 (A2)
- new net Rdh: C8.2, C9.2, R19.1
- new net VinP: C4.1, C5.1, C6.1, DZ1.1 (K), L1.1, Q1.2 (S), R1.1, TP1.1
Other:
- moved on the sheet: C10, C11, C3, C7, DZ1, J8, Q1, R4

Commit message: Update the title blocks
Other:
- company: (none) -> Hat Labs Oy
- title: (none) -> HALSPA - Hat Labs Spaghetti Board
Changed lines of the file:
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@@
 	(generator_version "9.0")
 	(paper "A4")
+	(title_block
+		(title "HALSPA - Hat Labs Spaghetti Board")
+		(date "2025-04-17")
+		(rev "v0.2.0")
+		(company "Hat Labs Oy")
+		(comment 1 "See the accompanying LICENSE.md file for license details.")
+	)
 	(text "0x20"
 		(exclude_from_sim no)
@@
 		(polyline
 			(pts
-				(xy 173.99 60.96) (xy 173.99 104.14) (xy 176.53 104.14) (xy 176.53 60.96)
+				(xy 137.16 68.58) (xy 137.16 59.69) (xy 134.62 59.69) (xy 134.62 68.58)
 			)
 			(stroke
@@
 		(polyline
 			(pts
-				(xy 137.16 68.58) (xy 137.16 59.69) (xy 134.62 59.69) (xy 134.62 68.58)
+				(xy 173.99 60.96) (xy 173.99 104.14) (xy 176.53 104.14) (xy 176.53 60.96)
 			)
 			(stroke

Commit message: Add JLCPCB corrections
Parts:
- D1, D11, D13, D15, D17, D19, D2, D4, D5, D7, D9: LCSC C2986059 -> C84267
- J10, J7, J9: JLCPCB_CORRECTION (none) -> 1.27;3.81;270
- J8: JLCPCB_CORRECTION (none) -> 1.905;0;0; now in the parts list
- U1: LCSC C22396388 -> C130204
Changed lines of the file:
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@@
 			)
 		)
-		(property "LCSC" "C2986059"
+		(property "LCSC" "C84267"
 			(at 113.03 138.43 0)
 			(effects
@@
 			)
 		)
-		(property "LCSC" "C2986059"
+		(property "LCSC" "C84267"
 			(at 153.67 138.43 0)
 			(effects
@@
 			)
 		)
+		(property "JLCPCB_CORRECTION" "1.27;3.81;270"
+			(at 66.04 127 0)
+			(effects
+				(font
+					(size 1.27 1.27)
+				)
+				(hide yes)
+			)
+		)
 		(pin "3"
 		)
@@
 			)
 		)
-		(property "LCSC" "C2986059"
+		(property "LCSC" "C84267"
 			(at 163.83 138.43 0)
 			(effects
@@
 			)
 		)
-		(property "LCSC Part" ""
-			(at 144.78 22.86 0)
-			(effects
-				(font
-					(size 1.27 1.27)
-				)
-			)
-		)
 		(property "Field8" ""
 			(at 144.78 22.86 0)
@@
 			)
 		)
+		(property "JLCPCB_CORRECTION" "1.27;3.81;270"
+			(at 45.72 127 0)
+			(effects
+				(font
+					(size 1.27 1.27)
+				)
+				(hide yes)
+			)
+		)
 		(pin "3"
 		)
@@
 			)
 		)
-		(property "LCSC Part" ""
-			(at 166.37 27.94 0)
-			(effects
-				(font
-					(size 1.27 1.27)
-				)
-			)
-		)
 		(property "Field8" ""
 			(at 166.37 27.94 0)
@@
 			)
 		)
-		(property "LCSC" "C2986059"
+		(property "LCSC" "C84267"
 			(at 133.35 138.43 0)
 			(effects
@@
 			)
 		)
-		(property "LCSC" "C2986059"
+		(property "LCSC" "C84267"
 			(at 104.14 138.43 0)
 			(effects
@@
 			)
 		)
-		(property "LCSC Part" ""
-			(at 156.21 27.94 0)
-			(effects
-				(font
-					(size 1.27 1.27)
-				)
-			)
-		)
 		(property "Field8" ""
 			(at 156.21 27.94 0)
@@
 			)
 		)
-		(property "LCSC Part" ""
-			(at 134.62 27.94 0)
-			(effects
-				(font
-					(size 1.27 1.27)
-				)
-			)
-		)
 		(property "Field8" ""
 			(at 134.62 27.94 0)
@@
 			)
 		)
-		(property "LCSC" "C2986059"
+		(property "LCSC" "C84267"
 			(at 60.96 171.45 0)
 			(effects
@@
 			)
 		)
-		(property "LCSC" "C2986059"
+		(property "LCSC" "C84267"
 			(at 31.75 171.45 0)
 			(effects
@@
 			)
 		)
-		(property "LCSC Part" ""
-			(at 110.49 27.94 0)
-			(effects
-				(font
-					(size 1.27 1.27)
-				)
-			)
-		)
 		(property "Field8" ""
 			(at 110.49 27.94 0)
@@
 			)
 		)
-		(property "LCSC" "C2986059"
+		(property "LCSC" "C84267"
 			(at 123.19 138.43 0)
 			(effects
@@
 			)
 		)
-		(property "LCSC" "C2986059"
+		(property "LCSC" "C84267"
 			(at 93.98 138.43 0)
 			(effects
@@
 			)
 		)
-		(property "LCSC Part" ""
-			(at 161.29 36.83 0)
-			(effects
-				(font
-					(size 1.27 1.27)
-				)
-			)
-		)
 		(property "Field8" ""
 			(at 161.29 36.83 0)
@@
 			)
 		)
-		(property "Datasheet" "https://www.lcsc.com/datasheet/lcsc_datasheet_2410010333_UMW-Youtai-Semiconductor-Co---Ltd--TCA9535PWR-UMW_C22396388.pdf"
+		(property "Datasheet" "https://www.ti.com/lit/ds/symlink/tca9535.pdf"
 			(at 143.51 59.69 0)
 			(effects
@@
 			)
 		)
-		(property "LCSC" "C22396388"
+		(property "LCSC" "C130204"
 			(at 156.21 82.55 0)
 			(effects
@@
 			)
 		)
+		(property "JLCPCB_CORRECTION" "1.27;3.81;270"
+			(at 25.4 127 0)
+			(effects
+				(font
+					(size 1.27 1.27)
+				)
+				(hide yes)
+			)
+		)
 		(pin "3"
 		)
@@
 			)
 		)
-		(property "LCSC" "C2986059"
+		(property "LCSC" "C84267"
 			(at 143.51 138.43 0)
 			(effects
@@
 		(unit 1)
 		(exclude_from_sim no)
-		(in_bom no)
+		(in_bom yes)
 		(on_board yes)
 		(dnp no)
@@
 			)
 		)
-		(property "JLCPCB_CORRECTION" ""
+		(property "JLCPCB_CORRECTION" "1.905;0;0"
 			(at 33.02 25.4 0)
 			(effects
@@
 			)
 		)
-		(property "LCSC" "C2986059"
+		(property "LCSC" "C84267"
 			(at 45.72 171.45 0)
 			(effects
@@
 			)
 		)
-		(property "LCSC Part" ""
-			(at 123.19 27.94 0)
-			(effects
-				(font
-					(size 1.27 1.27)
-				)
-			)
-		)
