File: adc.kicad_sch (KiCad schematic)
At the start: 0 parts

Commit message: WIP v0.2.0 changes
Other:
- sheet ADS1115 1 ports: added ALERT/RDY; removed none
- sheet ADS1115 2 ports: added ALERT/RDY; removed none
Changed lines of the file:
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@@
+	(wire
+		(pts
+			(xy 140.97 71.12) (xy 137.16 71.12)
+		)
+		(stroke
+			(width 0)
+			(type default)
+		)
+	)
 	(wire
 		(pts
@@
 			(width 0)
 			(type default)
+		)
+	)
+	(wire
+		(pts
+			(xy 140.97 38.1) (xy 137.16 38.1)
+		)
+		(stroke
+			(width 0)
+			(type default)
+		)
+	)
+	(hierarchical_label "ALERT1"
+		(shape output)
+		(at 140.97 38.1 0)
+		(effects
+			(font
+				(size 1.27 1.27)
+			)
+			(justify left)
+		)
+	)
+	(hierarchical_label "ALERT2"
+		(shape output)
+		(at 140.97 71.12 0)
+		(effects
+			(font
+				(size 1.27 1.27)
+			)
+			(justify left)
 		)
 	)
@@
 		(dnp no)
 		(fields_autoplaced yes)
-		(property "Reference" "#PWR0157"
+		(property "Reference" "#PWR0154"
 			(at 96.52 86.36 0)
 			(effects
@@
 			(project ""
 				(path "/7eeba806-440e-4671-bc07-69fe183910a7/f863d577-5163-4667-a0b3-93abcffbcf80"
-					(reference "#PWR0157")
+					(reference "#PWR0154")
 					(unit 1)
 				)
@@
 		(dnp no)
 		(fields_autoplaced yes)
-		(property "Reference" "#PWR0156"
+		(property "Reference" "#PWR0153"
 			(at 96.52 58.42 0)
 			(effects
@@
 			(project ""
 				(path "/7eeba806-440e-4671-bc07-69fe183910a7/f863d577-5163-4667-a0b3-93abcffbcf80"
-					(reference "#PWR0156")
+					(reference "#PWR0153")
 					(unit 1)
 				)
@@
 				)
 				(justify left)
+			)
+		)
+		(pin "ALERT{slash}RDY" output
+			(at 137.16 71.12 0)
+			(effects
+				(font
+					(size 1.27 1.27)
+				)
+				(justify right)
 			)
 		)
@@
 			)
 		)
+		(pin "ALERT{slash}RDY" output
+			(at 137.16 38.1 0)
+			(effects
+				(font
+					(size 1.27 1.27)
+				)
+				(justify right)
+			)
+		)

Commit message: Update the title blocks
Other:
- company: (none) -> Hat Labs Oy
- title: (none) -> HALSPA - Hat Labs Spaghetti Board
Changed lines of the file:
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@@
 	(generator_version "9.0")
 	(paper "A4")
+	(title_block
+		(title "HALSPA - Hat Labs Spaghetti Board")
+		(date "2025-04-17")
+		(rev "v0.2.0")
+		(company "Hat Labs Oy")
+		(comment 1 "See the accompanying LICENSE.md file for license details.")
+	)
 	(text "0x48"
 		(exclude_from_sim no)
