File: anaio.kicad_sch (KiCad schematic)
At the start: 8 parts, among them J42 Conn_01x04, J43 Conn_01x02, J44 Conn_01x02, J45 Conn_01x04, J46 Conn_01x02, J47 Conn_01x02, U23 TCA9535PWR(UMW)

Commit message: Update the design to a stackable one
Parts:
- removed J42, J45: Conn_01x04, HL_Connector_Pad_2.54mm:Pad_1x04_P2.54_1.7x1.7_Rect, symbol Connector_Generic:Conn_01x04
- removed J43, J44, J46, J47: Conn_01x02, HL_Connector_Pad_2.54mm:Pad_1x02_P2.54_1.7x1.7_Rect-Rnd, symbol Connector_Generic:Conn_01x02
- renumbered C51 to C61
Other:
- sheet Analog MUX 1 ports: added none; removed D
- sheet Analog MUX 2 ports: added none; removed D
- sheet Analog MUX 3 ports: added none; removed D
- sheet Analog MUX 4 ports: added none; removed D
