File: buck_3.3V.kicad_sch (KiCad schematic)
At the start: 14 parts, among them U2 TPS566238PRQFR

Commit message: WIP v0.2.0 changes
Parts:
- added R80: 10k, Resistor_SMD:R_0603_1608Metric_Pad0.98x0.95mm_HandSolder, symbol Device:R_Small
Connections:
- net EN: now also R80.1
- net GND: now also R80.2
Changed lines of the file:
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@@
+	(wire
+		(pts
+			(xy 100.33 121.92) (xy 100.33 116.84)
+		)
+		(stroke
+			(width 0)
+			(type default)
+		)
+	)
 	(wire
 		(pts
@@
 	(wire
 		(pts
+			(xy 100.33 127) (xy 100.33 130.81)
+		)
+		(stroke
+			(width 0)
+			(type default)
+		)
+	)
+	(wire
+		(pts
 			(xy 233.68 77.47) (xy 233.68 78.74)
 		)
@@
 		(pts
 			(xy 194.31 80.01) (xy 194.31 85.09)
+		)
+		(stroke
+			(width 0)
+			(type default)
+		)
+	)
+	(wire
+		(pts
+			(xy 100.33 116.84) (xy 97.79 116.84)
 		)
 		(stroke
@@
 		(shape input)
 		(at 48.26 62.23 180)
+		(effects
+			(font
+				(size 1.27 1.27)
+			)
+			(justify right)
+		)
+	)
+	(hierarchical_label "EN"
+		(shape input)
+		(at 97.79 116.84 180)
 		(effects
 			(font
@@
 		(on_board yes)
 		(dnp no)
-		(property "Reference" "#PWR059"
+		(property "Reference" "#PWR058"
 			(at 71.12 88.9 0)
 			(effects
@@
 			(project "HALSPA"
 				(path "/7eeba806-440e-4671-bc07-69fe183910a7/8a7bd3c3-3783-4a08-9c22-bb373aae5663/b99533d9-3b4f-461f-95f4-04c4f9d347c7"
-					(reference "#PWR059")
+					(reference "#PWR058")
 					(unit 1)
 				)
@@
 		(on_board yes)
 		(dnp no)
-		(property "Reference" "#PWR063"
+		(property "Reference" "#PWR062"
 			(at 194.31 91.44 0)
 			(effects
@@
 			(project "HALSPA"
 				(path "/7eeba806-440e-4671-bc07-69fe183910a7/8a7bd3c3-3783-4a08-9c22-bb373aae5663/b99533d9-3b4f-461f-95f4-04c4f9d347c7"
-					(reference "#PWR063")
+					(reference "#PWR062")
 					(unit 1)
 				)
@@
 		(on_board yes)
 		(dnp no)
-		(property "Reference" "#PWR064"
+		(property "Reference" "#PWR063"
 			(at 212.09 91.44 0)
 			(effects
@@
 			(project "HALSPA"
 				(path "/7eeba806-440e-4671-bc07-69fe183910a7/8a7bd3c3-3783-4a08-9c22-bb373aae5663/b99533d9-3b4f-461f-95f4-04c4f9d347c7"
-					(reference "#PWR064")
+					(reference "#PWR063")
 					(unit 1)
 				)
@@
 		(on_board yes)
 		(dnp no)
-		(property "Reference" "#PWR062"
+		(property "Reference" "#PWR061"
 			(at 182.88 91.44 0)
 			(effects
@@
 			(project "HALSPA"
 				(path "/7eeba806-440e-4671-bc07-69fe183910a7/8a7bd3c3-3783-4a08-9c22-bb373aae5663/b99533d9-3b4f-461f-95f4-04c4f9d347c7"
-					(reference "#PWR062")
+					(reference "#PWR061")
 					(unit 1)
 				)
@@
 	)
 	(symbol
+		(lib_id "Device:R_Small")
+		(at 100.33 124.46 0)
+		(unit 1)
+		(exclude_from_sim no)
+		(in_bom yes)
+		(on_board yes)
+		(dnp no)
+		(fields_autoplaced yes)
+		(property "Reference" "R80"
+			(at 102.87 123.1899 0)
+			(effects
+				(font
+					(size 1.016 1.016)
+				)
+				(justify left)
+			)
+		)
+		(property "Value" "10k"
+			(at 102.87 125.7299 0)
+			(effects
+				(font
+					(size 1.27 1.27)
+				)
+				(justify left)
+			)
+		)
+		(property "Footprint" "Resistor_SMD:R_0603_1608Metric_Pad0.98x0.95mm_HandSolder"
+			(at 100.33 124.46 0)
+			(effects
+				(font
+					(size 1.27 1.27)
+				)
+				(hide yes)
+			)
+		)
+		(property "Datasheet" "~"
+			(at 100.33 124.46 0)
+			(effects
+				(font
+					(size 1.27 1.27)
+				)
+				(hide yes)
+			)
+		)
+		(property "Description" "Resistor, small symbol"
+			(at 100.33 124.46 0)
+			(effects
+				(font
+					(size 1.27 1.27)
+				)
+				(hide yes)
+			)
+		)
+		(property "LCSC" "C25804"
+			(at 100.33 124.46 0)
+			(effects
+				(font
+					(size 1.27 1.27)
+				)
+			)
+		)
+		(pin "1"
+		)
+		(pin "2"
+		)
+		(instances
+			(project "HALSPA"
+				(path "/7eeba806-440e-4671-bc07-69fe183910a7/8a7bd3c3-3783-4a08-9c22-bb373aae5663/b99533d9-3b4f-461f-95f4-04c4f9d347c7"
+					(reference "R80")
+					(unit 1)
+				)
+			)
+		)
+	)
+	(symbol
 		(lib_id "Device:R")
 		(at 95.25 82.55 270)
@@
 		(on_board yes)
 		(dnp no)
-		(property "Reference" "#PWR058"
+		(property "Reference" "#PWR057"
 			(at 57.15 88.9 0)
 			(effects
@@
 			(project "HALSPA"
 				(path "/7eeba806-440e-4671-bc07-69fe183910a7/8a7bd3c3-3783-4a08-9c22-bb373aae5663/b99533d9-3b4f-461f-95f4-04c4f9d347c7"
-					(reference "#PWR058")
+					(reference "#PWR057")
 					(unit 1)
 				)
@@
 		(on_board yes)
 		(dnp no)
-		(property "Reference" "#PWR065"
+		(property "Reference" "#PWR064"
 			(at 222.25 96.52 0)
 			(effects
@@
 			(project "HALSPA"
 				(path "/7eeba806-440e-4671-bc07-69fe183910a7/8a7bd3c3-3783-4a08-9c22-bb373aae5663/b99533d9-3b4f-461f-95f4-04c4f9d347c7"
-					(reference "#PWR065")
+					(reference "#PWR064")
 					(unit 1)
 				)
@@
 		(on_board yes)
 		(dnp no)
-		(property "Reference" "#PWR060"
+		(property "Reference" "#PWR059"
 			(at 87.63 104.14 0)
 			(effects
@@
 			(project "HALSPA"
 				(path "/7eeba806-440e-4671-bc07-69fe183910a7/8a7bd3c3-3783-4a08-9c22-bb373aae5663/b99533d9-3b4f-461f-95f4-04c4f9d347c7"
-					(reference "#PWR060")
+					(reference "#PWR059")
 					(unit 1)
 				)
@@
 		(on_board yes)
 		(dnp no)
-		(property "Reference" "#PWR061"
+		(property "Reference" "#PWR060"
 			(at 123.19 104.14 0)
 			(effects
@@
 			(project "HALSPA"
 				(path "/7eeba806-440e-4671-bc07-69fe183910a7/8a7bd3c3-3783-4a08-9c22-bb373aae5663/b99533d9-3b4f-461f-95f4-04c4f9d347c7"
-					(reference "#PWR061")
+					(reference "#PWR060")
 					(unit 1)
 				)
@@
 					(unit 1)
 				)
+			)
+		)
+	)
+	(symbol
+		(lib_id "power:GND")
+		(at 100.33 130.81 0)
+		(mirror y)
+		(unit 1)
+		(exclude_from_sim no)
+		(in_bom yes)
+		(on_board yes)
+		(dnp no)
+		(fields_autoplaced yes)
+		(property "Reference" "#PWR0229"
+			(at 100.33 137.16 0)
+			(effects
+				(font
+					(size 1.27 1.27)
+				)
+				(hide yes)
+			)
+		)
+		(property "Value" "GND"
+			(at 100.33 135.89 0)
+			(effects
+				(font
+					(size 1.27 1.27)
+				)
+			)
+		)
+		(property "Footprint" ""
+			(at 100.33 130.81 0)
+			(effects
+				(font
+					(size 1.27 1.27)
+				)
+				(hide yes)
+			)
+		)
+		(property "Datasheet" ""
+			(at 100.33 130.81 0)
+			(effects
+				(font
+					(size 1.27 1.27)
+				)
+				(hide yes)
+			)
+		)
+		(property "Description" "Power symbol creates a global label with name \"GND\" , ground"
+			(at 100.33 130.81 0)
+			(effects
+				(font
+					(size 1.27 1.27)
+				)
+				(hide yes)
+			)
+		)
+		(pin "1"
+		)
+		(instances
+			(project "HALSPA"
+				(path "/7eeba806-440e-4671-bc07-69fe183910a7/8a7bd3c3-3783-4a08-9c22-bb373aae5663/b99533d9-3b4f-461f-95f4-04c4f9d347c7"
+					(reference "#PWR0229")
+					(unit 1)
+				)

Commit message: Assign part numbers and finish other 0.2.0 changes
Parts:
- renumbered C7 to C12, C8 to C13, C9 to C14, C10 to C15, C11 to C16, C12 to C17, C13 to C18, C14 to C19, L1 to L2, R21 to R22, R80 to R23, R22 to R24, R23 to R25, TP1 to TP2
Changed lines of the file:
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@@
 		(on_board yes)
 		(dnp no)
-		(property "Reference" "#PWR058"
+		(property "Reference" "#PWR063"
 			(at 71.12 88.9 0)
 			(effects
@@
 			(project "HALSPA"
 				(path "/7eeba806-440e-4671-bc07-69fe183910a7/8a7bd3c3-3783-4a08-9c22-bb373aae5663/b99533d9-3b4f-461f-95f4-04c4f9d347c7"
-					(reference "#PWR058")
+					(reference "#PWR063")
 					(unit 1)
 				)
@@
 		(on_board yes)
 		(dnp no)
-		(property "Reference" "#PWR062"
+		(property "Reference" "#PWR068"
 			(at 194.31 91.44 0)
 			(effects
@@
 			(project "HALSPA"
 				(path "/7eeba806-440e-4671-bc07-69fe183910a7/8a7bd3c3-3783-4a08-9c22-bb373aae5663/b99533d9-3b4f-461f-95f4-04c4f9d347c7"
-					(reference "#PWR062")
+					(reference "#PWR068")
 					(unit 1)
 				)
@@
 		(on_board yes)
 		(dnp no)
-		(property "Reference" "#PWR063"
+		(property "Reference" "#PWR069"
 			(at 212.09 91.44 0)
 			(effects
@@
 			(project "HALSPA"
 				(path "/7eeba806-440e-4671-bc07-69fe183910a7/8a7bd3c3-3783-4a08-9c22-bb373aae5663/b99533d9-3b4f-461f-95f4-04c4f9d347c7"
-					(reference "#PWR063")
+					(reference "#PWR069")
 					(unit 1)
 				)
@@
 		(dnp no)
 		(fields_autoplaced yes)
-		(property "Reference" "C14"
+		(property "Reference" "C19"
 			(at 237.49 72.3899 0)
 			(effects
@@
 			(project "HALSPA"
 				(path "/7eeba806-440e-4671-bc07-69fe183910a7/8a7bd3c3-3783-4a08-9c22-bb373aae5663/b99533d9-3b4f-461f-95f4-04c4f9d347c7"
-					(reference "C14")
+					(reference "C19")
 					(unit 1)
 				)
@@
 		(on_board yes)
 		(dnp no)
-		(property "Reference" "#PWR061"
+		(property "Reference" "#PWR067"
 			(at 182.88 91.44 0)
 			(effects
@@
 			(project "HALSPA"
 				(path "/7eeba806-440e-4671-bc07-69fe183910a7/8a7bd3c3-3783-4a08-9c22-bb373aae5663/b99533d9-3b4f-461f-95f4-04c4f9d347c7"
-					(reference "#PWR061")
+					(reference "#PWR067")
 					(unit 1)
 				)
@@
 		(on_board yes)
 		(dnp no)
-		(property "Reference" "C10"
+		(property "Reference" "C15"
 			(at 166.37 55.88 90)
 			(effects
@@
 			(project "HALSPA"
 				(path "/7eeba806-440e-4671-bc07-69fe183910a7/8a7bd3c3-3783-4a08-9c22-bb373aae5663/b99533d9-3b4f-461f-95f4-04c4f9d347c7"
-					(reference "C10")
+					(reference "C15")
 					(unit 1)
 				)
@@
 		(on_board yes)
 		(dnp no)
-		(property "Reference" "TP1"
+		(property "Reference" "TP2"
 			(at 242.57 80.7719 0)
 			(effects
@@
 			(project "HALSPA"
 				(path "/7eeba806-440e-4671-bc07-69fe183910a7/8a7bd3c3-3783-4a08-9c22-bb373aae5663/b99533d9-3b4f-461f-95f4-04c4f9d347c7"
-					(reference "TP1")
+					(reference "TP2")
 					(unit 1)
 				)
@@
 		(dnp no)
 		(fields_autoplaced yes)
-		(property "Reference" "R22"
+		(property "Reference" "R24"
 			(at 224.79 72.3899 0)
 			(effects
@@
 			(project "HALSPA"
 				(path "/7eeba806-440e-4671-bc07-69fe183910a7/8a7bd3c3-3783-4a08-9c22-bb373aae5663/b99533d9-3b4f-461f-95f4-04c4f9d347c7"
-					(reference "R22")
+					(reference "R24")
 					(unit 1)
 				)
@@
 		(on_board yes)
 		(dnp no)
-		(property "Reference" "C8"
+		(property "Reference" "C13"
 			(at 68.199 69.9516 0)
 			(effects
@@
 			(project "HALSPA"
 				(path "/7eeba806-440e-4671-bc07-69fe183910a7/8a7bd3c3-3783-4a08-9c22-bb373aae5663/b99533d9-3b4f-461f-95f4-04c4f9d347c7"
-					(reference "C8")
+					(reference "C13")
 					(unit 1)
 				)
@@
 		(on_board yes)
 		(dnp no)
-		(property "Reference" "C11"
+		(property "Reference" "C16"
 			(at 179.959 78.8416 0)
 			(effects
@@
 			(project "HALSPA"
 				(path "/7eeba806-440e-4671-bc07-69fe183910a7/8a7bd3c3-3783-4a08-9c22-bb373aae5663/b99533d9-3b4f-461f-95f4-04c4f9d347c7"
-					(reference "C11")
+					(reference "C16")
 					(unit 1)
 				)
@@
 		(dnp no)
 		(fields_autoplaced yes)
-		(property "Reference" "R23"
+		(property "Reference" "R25"
 			(at 224.79 83.8199 0)
 			(effects
@@
 			(project "HALSPA"
 				(path "/7eeba806-440e-4671-bc07-69fe183910a7/8a7bd3c3-3783-4a08-9c22-bb373aae5663/b99533d9-3b4f-461f-95f4-04c4f9d347c7"
-					(reference "R23")
+					(reference "R25")
 					(unit 1)
 				)
@@
 		(dnp no)
 		(fields_autoplaced yes)
-		(property "Reference" "R80"
+		(property "Reference" "R23"
 			(at 102.87 123.1899 0)
 			(effects
@@
 			(project "HALSPA"
 				(path "/7eeba806-440e-4671-bc07-69fe183910a7/8a7bd3c3-3783-4a08-9c22-bb373aae5663/b99533d9-3b4f-461f-95f4-04c4f9d347c7"
-					(reference "R80")
+					(reference "R23")
 					(unit 1)
 				)
@@
 		(on_board yes)
 		(dnp no)
-		(property "Reference" "R21"
+		(property "Reference" "R22"
 			(at 95.25 85.344 90)
 			(effects
@@
 			(project "HALSPA"
 				(path "/7eeba806-440e-4671-bc07-69fe183910a7/8a7bd3c3-3783-4a08-9c22-bb373aae5663/b99533d9-3b4f-461f-95f4-04c4f9d347c7"
-					(reference "R21")
+					(reference "R22")
 					(unit 1)
 				)
@@
 		(on_board yes)
 		(dnp no)
-		(property "Reference" "#PWR057"
+		(property "Reference" "#PWR062"
 			(at 57.15 88.9 0)
 			(effects
@@
 			(project "HALSPA"
 				(path "/7eeba806-440e-4671-bc07-69fe183910a7/8a7bd3c3-3783-4a08-9c22-bb373aae5663/b99533d9-3b4f-461f-95f4-04c4f9d347c7"
-					(reference "#PWR057")
+					(reference "#PWR062")
 					(unit 1)
 				)
@@
 		(on_board yes)
 		(dnp no)
-		(property "Reference" "#PWR064"
+		(property "Reference" "#PWR070"
 			(at 222.25 96.52 0)
 			(effects
@@
 			(project "HALSPA"
 				(path "/7eeba806-440e-4671-bc07-69fe183910a7/8a7bd3c3-3783-4a08-9c22-bb373aae5663/b99533d9-3b4f-461f-95f4-04c4f9d347c7"
-					(reference "#PWR064")
+					(reference "#PWR070")
 					(unit 1)
 				)
@@
 		(on_board yes)
 		(dnp no)
-		(property "Reference" "C13"
+		(property "Reference" "C18"
 			(at 209.169 72.4916 0)
 			(effects
@@
 			(project "HALSPA"
 				(path "/7eeba806-440e-4671-bc07-69fe183910a7/8a7bd3c3-3783-4a08-9c22-bb373aae5663/b99533d9-3b4f-461f-95f4-04c4f9d347c7"
-					(reference "C13")
+					(reference "C18")
 					(unit 1)
 				)
@@
 		(on_board yes)
 		(dnp no)
-		(property "Reference" "C7"
+		(property "Reference" "C12"
 			(at 54.229 69.9516 0)
 			(effects
@@
 			(project "HALSPA"
 				(path "/7eeba806-440e-4671-bc07-69fe183910a7/8a7bd3c3-3783-4a08-9c22-bb373aae5663/b99533d9-3b4f-461f-95f4-04c4f9d347c7"
-					(reference "C7")
+					(reference "C12")
 					(unit 1)
 				)
@@
 		(on_board yes)
 		(dnp no)
-		(property "Reference" "#PWR059"
+		(property "Reference" "#PWR064"
 			(at 87.63 104.14 0)
 			(effects
@@
 			(project "HALSPA"
 				(path "/7eeba806-440e-4671-bc07-69fe183910a7/8a7bd3c3-3783-4a08-9c22-bb373aae5663/b99533d9-3b4f-461f-95f4-04c4f9d347c7"
-					(reference "#PWR059")
+					(reference "#PWR064")
 					(unit 1)
 				)
@@
 		(on_board yes)
 		(dnp no)
-		(property "Reference" "#PWR060"
+		(property "Reference" "#PWR066"
 			(at 123.19 104.14 0)
 			(effects
@@
 			(project "HALSPA"
 				(path "/7eeba806-440e-4671-bc07-69fe183910a7/8a7bd3c3-3783-4a08-9c22-bb373aae5663/b99533d9-3b4f-461f-95f4-04c4f9d347c7"
-					(reference "#PWR060")
+					(reference "#PWR066")
 					(unit 1)
 				)
@@
 		(on_board yes)
 		(dnp no)
-		(property "Reference" "C12"
+		(property "Reference" "C17"
 			(at 191.389 75.0316 0)
 			(effects
@@
 			(project "HALSPA"
 				(path "/7eeba806-440e-4671-bc07-69fe183910a7/8a7bd3c3-3783-4a08-9c22-bb373aae5663/b99533d9-3b4f-461f-95f4-04c4f9d347c7"
-					(reference "C12")
+					(reference "C17")
 					(unit 1)
 				)
@@
 		(dnp no)
 		(fields_autoplaced yes)
-		(property "Reference" "#FLG06"
+		(property "Reference" "#FLG07"
 			(at 207.01 65.405 0)
 			(effects
@@
 			(project "HALSPA"
 				(path "/7eeba806-440e-4671-bc07-69fe183910a7/8a7bd3c3-3783-4a08-9c22-bb373aae5663/b99533d9-3b4f-461f-95f4-04c4f9d347c7"
-					(reference "#FLG06")
+					(reference "#FLG07")
 					(unit 1)
 				)
@@
 		(on_board yes)
 		(dnp no)
-		(property "Reference" "L1"
+		(property "Reference" "L2"
 			(at 175.26 62.484 90)
 			(effects
@@
 			(project "HALSPA"
 				(path "/7eeba806-440e-4671-bc07-69fe183910a7/8a7bd3c3-3783-4a08-9c22-bb373aae5663/b99533d9-3b4f-461f-95f4-04c4f9d347c7"
-					(reference "L1")
+					(reference "L2")
 					(unit 1)
 				)
@@
 		(dnp no)
 		(fields_autoplaced yes)
-		(property "Reference" "#PWR0229"
+		(property "Reference" "#PWR065"
 			(at 100.33 137.16 0)
 			(effects
@@
 			(project "HALSPA"
 				(path "/7eeba806-440e-4671-bc07-69fe183910a7/8a7bd3c3-3783-4a08-9c22-bb373aae5663/b99533d9-3b4f-461f-95f4-04c4f9d347c7"
-					(reference "#PWR0229")
+					(reference "#PWR065")
 					(unit 1)
 				)
@@
 		(on_board yes)
 		(dnp no)
-		(property "Reference" "C9"
+		(property "Reference" "C14"
 			(at 84.709 90.2716 0)
 			(effects
@@
 			(project "HALSPA"
 				(path "/7eeba806-440e-4671-bc07-69fe183910a7/8a7bd3c3-3783-4a08-9c22-bb373aae5663/b99533d9-3b4f-461f-95f4-04c4f9d347c7"
-					(reference "C9")
-					(unit 1)
-				)
+					(reference "C14")
+					(unit 1)
+				)

Commit message: Update the title blocks
Other:
- title: HALPI2 -> HALSPA - Hat Labs Spaghetti Board
Changed lines of the file:
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@@
 	(paper "A4")
 	(title_block
-		(title "HALPI2")
-		(date "2025-01-26")
-		(rev "v0.0.1")
+		(title "HALSPA - Hat Labs Spaghetti Board")
+		(date "2025-04-17")
+		(rev "v0.2.0")
 		(company "Hat Labs Oy")
-		(comment 1 "https://ohwr.org/cern_ohl_s_v2.pdf")
+		(comment 1 "See the accompanying LICENSE.md file for license details.")
 		(comment 2 "To view a copy of this license, visit ")
 		(comment 3 "HALPI2 is licensed under CERN-OHL-S v2.")

Commit message: Update the design to a stackable one
Parts:
- removed TP2: FB3, TestPoint:TestPoint_Pad_D1.0mm, symbol Connector:TestPoint
- added D5: GREEN, LED_SMD:LED_0603_1608Metric, symbol Device:LED
- added D6: RED, LED_SMD:LED_0603_1608Metric, symbol Device:LED
- added R10: 1.5k, Resistor_SMD:R_0603_1608Metric, symbol Device:R
- added R11: 2k, Resistor_SMD:R_0603_1608Metric, symbol Device:R
- renumbered R24 to R12, R25 to R13, R22 to R8, R23 to R9
Connections:
- net EN: now also R10.1, R11.1
- net GND: now also D5.1 (K)
- new net: D5.2 (A), R10.2
- new net: D6.2 (A), R11.2
- new net +3.3VD: D6.1 (K)
