File: current_sense.kicad_sch (KiCad schematic)
At the start: 0 parts

Commit message: Update the title blocks
Other:
- company: (none) -> Hat Labs Oy
- title: (none) -> HALSPA - Hat Labs Spaghetti Board
Changed lines of the file:
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@@
 	(generator_version "9.0")
 	(paper "A4")
+	(title_block
+		(title "HALSPA - Hat Labs Spaghetti Board")
+		(date "2025-04-17")
+		(rev "v0.2.0")
+		(company "Hat Labs Oy")
+		(comment 1 "See the accompanying LICENSE.md file for license details.")
+	)
 	(sheet
 		(at 57.15 128.27)
