File: digio.kicad_sch (KiCad schematic)
At the start: 42 parts, among them J25 Conn_01x08, J26 Conn_01x08, J27 Conn_01x08, J28 Conn_01x08, J29 Conn_01x04, J30 Conn_01x04, U18 TCA9535PWR(UMW), U19 TCA9535PWR(UMW)

Commit message: Assorted fixes
Connections:
- net P1r00: now also R62.2; no longer R46.2
- net P1r01: now also R63.2; no longer R47.2
- net P1r02: now also R64.2; no longer R48.2
- net P1r03: now also R65.2; no longer R49.2
- net P1r04: now also R66.2; no longer R50.2
- net P1r05: now also R67.2; no longer R51.2
- net P1r06: now also R68.2; no longer R52.2
- net P1r07: now also R69.2; no longer R53.2
- net P1r10: now also R70.2; no longer R54.2
- net P1r11: now also R71.2; no longer R55.2
- net P1r12: now also R72.2; no longer R56.2
- net P1r13: now also R73.2; no longer R57.2
- net P1r14: now also R74.2; no longer R58.2
- net P1r15: now also R75.2; no longer R59.2
- net P1r16: now also R76.2; no longer R60.2
- net P1r17: now also R77.2; no longer R61.2
- net P2r00: now also R46.2; no longer R62.2
- net P2r01: now also R47.2; no longer R63.2
- net P2r02: now also R48.2; no longer R64.2
- net P2r03: now also R49.2; no longer R65.2
- net P2r04: now also R50.2; no longer R66.2
- net P2r05: now also R51.2; no longer R67.2
- net P2r06: now also R52.2; no longer R68.2
- net P2r07: now also R53.2; no longer R69.2
- net P2r10: now also R54.2; no longer R70.2
- net P2r11: now also R55.2; no longer R71.2
- net P2r12: now also R56.2; no longer R72.2
- net P2r13: now also R57.2; no longer R73.2
- net P2r14: now also R58.2; no longer R74.2
- net P2r15: now also R59.2; no longer R75.2
- net P2r16: now also R60.2; no longer R76.2
- net P2r17: now also R61.2; no longer R77.2
Other:
- moved on the sheet: C46, C47, J25, J26, J27, J28, J29, J30, R46, R47, R48, R49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

Commit message: Update the design to a stackable one
Parts:
- removed J29, J30: Conn_01x04, HL_Connector_Pad_2.54mm:Pad_1x04_P2.54_1.7x1.7_Rect, symbol Connector_Generic:Conn_01x04
- added JP1, JP10, JP11, JP12, JP13, JP14, JP15, JP16, JP17, JP18, JP19, JP2, JP20, JP21, JP22, JP23, JP24, JP25, JP26, JP27, JP28, JP29, JP3, JP30, JP31, JP32, JP4, JP5, JP6, JP7, JP8, JP9: SolderJumper_2_Open, Jumper:SolderJumper-2_P1.3mm_Open_TrianglePad1.0x1.5mm, symbol Jumper:SolderJumper_2_Open
- J18: renamed from J25; value Conn_01x08 -> Conn_02x05_Pin; footprint HL_Connector_Pad_2.54mm:Pad_1x08_P2.54_1.7x1.7_Oct -> HL_Connector_Pad_2.54mm:Pad_2x05_P2.54_1.7x1.7_2Rect-8Oct; symbol Connector_Generic:Conn_01x08 -> Connector_Generic:Conn_02x05_Odd_Even; JLCPCB_CORRECTION 0;8.89;270 -> 1.27;-5.08;270; LCSC C492407 -> C492422
- J19: renamed from J26; value Conn_01x08 -> Conn_02x05_Pin; footprint HL_Connector_Pad_2.54mm:Pad_1x08_P2.54_1.7x1.7_Oct -> HL_Connector_Pad_2.54mm:Pad_2x05_P2.54_1.7x1.7_2Rect-8Oct; symbol Connector_Generic:Conn_01x08 -> Connector_Generic:Conn_02x05_Odd_Even; JLCPCB_CORRECTION 0;8.89;270 -> 1.27;-5.08;270; LCSC C492407 -> C492422
- J20: renamed from J27; value Conn_01x08 -> Conn_02x05_Pin; footprint HL_Connector_Pad_2.54mm:Pad_1x08_P2.54_1.7x1.7_Oct -> HL_Connector_Pad_2.54mm:Pad_2x05_P2.54_1.7x1.7_2Rect-8Oct; symbol Connector_Generic:Conn_01x08 -> Connector_Generic:Conn_02x05_Odd_Even; JLCPCB_CORRECTION 0;8.89;270 -> 1.27;-5.08;270; LCSC C492407 -> C492422
- J21: renamed from J28; value Conn_01x08 -> Conn_02x05_Pin; footprint HL_Connector_Pad_2.54mm:Pad_1x08_P2.54_1.7x1.7_Oct -> HL_Connector_Pad_2.54mm:Pad_2x05_P2.54_1.7x1.7_2Rect-8Oct; symbol Connector_Generic:Conn_01x08 -> Connector_Generic:Conn_02x05_Odd_Even; JLCPCB_CORRECTION 0;8.89;270 -> 1.27;-5.08;270; LCSC C492407 -> C492422
- renumbered C47 to C48, C46 to C49, R62 to R50, R63 to R51, R64 to R52, R65 to R53, R66 to R54, R67 to R55, R68 to R56, R69 to R57, R70 to R58, R71 to R59, R72 to R60, R73 to R61, R74 to R62, R75 to R63, R76 to R64, R77 to R65, R46 to R66, R47 to R67, R48 to R68, R49 to R69, R50 to R70, R51 to R71, R52 to R72, R53 to R73, R54 to R74, R55 to R75, R56 to R76, R57 to R77, R58 to R78, R59 to R79, R60 to R80, R61 to R81, U19 to U18, U18 to U19
Connections:
- net GND: now also J18.3 (Pin_3), J18.8 (Pin_8), J19.3 (Pin_3), J19.8 (Pin_8), J20.3 (Pin_3), J20.8 (Pin_8), J21.3 (Pin_3), J21.8 (Pin_8)
- net P100: now also JP17.1 (A)
- net P101: now also JP18.1 (A)
- net P102: now also JP19.1 (A)
- net P103: now also JP20.1 (A)
- net P104: now also JP21.1 (A)
- net P105: now also JP22.1 (A)
- net P106: now also JP23.1 (A)
- net P107: now also JP24.1 (A)
- net P110: now also JP25.1 (A)
- net P111: now also JP26.1 (A)
- net P112: now also JP27.1 (A)
- net P113: now also JP28.1 (A)
- net P114: now also JP29.1 (A)
- net P115: now also JP30.1 (A)
- net P116: now also JP31.1 (A)
- net P117: now also JP32.1 (A)
- net P1r00: now also JP1.2 (B)
- net P1r01: now also JP2.2 (B)
- net P1r02: now also J18.4 (Pin_4), JP3.2 (B); no longer J18.3 (Pin_3)
- net P1r03: now also J18.6 (Pin_6), JP4.2 (B); no longer J18.4 (Pin_4)
- net P1r04: now also JP5.2 (B)
- net P1r05: now also J18.7 (Pin_7), JP6.2 (B); no longer J18.6 (Pin_6)
- net P1r06: now also J18.9 (Pin_9), JP7.2 (B); no longer J18.7 (Pin_7)
- net P1r07: now also J18.10 (Pin_10), JP8.2 (B); no longer J18.8 (Pin_8)
- net P1r10: now also J19.1 (Pin_1), JP9.2 (B); no longer J19.8 (Pin_8)
- net P1r11: now also J19.2 (Pin_2), JP10.2 (B); no longer J19.7 (Pin_7)
- net P1r12: now also J19.4 (Pin_4), JP11.2 (B); no longer J19.6 (Pin_6)
- net P1r13: now also J19.6 (Pin_6), JP12.2 (B); no longer J19.5 (Pin_5)
- net P1r14: now also J19.5 (Pin_5), JP13.2 (B); no longer J19.4 (Pin_4)
- net P1r15: now also J19.7 (Pin_7), JP14.2 (B); no longer J19.3 (Pin_3)
- net P1r16: now also J19.9 (Pin_9), JP15.2 (B); no longer J19.2 (Pin_2)
- net P1r17: now also J19.10 (Pin_10), JP16.2 (B); no longer J19.1 (Pin_1)
- net P200: now also JP1.1 (A)
- net P201: now also JP2.1 (A)
- net P202: now also JP3.1 (A)
- net P203: now also JP4.1 (A)
- net P204: now also JP5.1 (A)
- net P205: now also JP6.1 (A)
- net P206: now also JP7.1 (A)
- net P207: now also JP8.1 (A)
- net P210: now also JP9.1 (A)
- net P211: now also JP10.1 (A)
- net P212: now also JP11.1 (A)
- net P213: now also JP12.1 (A)
- net P214: now also JP13.1 (A)
- net P215: now also JP14.1 (A)
- net P216: now also JP15.1 (A)
- net P217: now also JP16.1 (A)
- net P2r00: now also JP17.2 (B)
- net P2r01: now also JP18.2 (B)
- net P2r02: now also J20.4 (Pin_4), JP19.2 (B); no longer J20.3 (Pin_3)
- net P2r03: now also J20.6 (Pin_6), JP20.2 (B); no longer J20.4 (Pin_4)
- net P2r04: now also JP21.2 (B)
- net P2r05: now also J20.7 (Pin_7), JP22.2 (B); no longer J20.6 (Pin_6)
- net P2r06: now also J20.9 (Pin_9), JP23.2 (B); no longer J20.7 (Pin_7)
- net P2r07: now also J20.10 (Pin_10), JP24.2 (B); no longer J20.8 (Pin_8)
- net P2r10: now also J21.1 (Pin_1), JP25.2 (B); no longer J21.8 (Pin_8)
- net P2r11: now also J21.2 (Pin_2), JP26.2 (B); no longer J21.7 (Pin_7)
- net P2r12: now also J21.4 (Pin_4), JP27.2 (B); no longer J21.6 (Pin_6)
- net P2r13: now also J21.6 (Pin_6), JP28.2 (B); no longer J21.5 (Pin_5)
- net P2r14: now also J21.5 (Pin_5), JP29.2 (B); no longer J21.4 (Pin_4)
- net P2r15: now also J21.7 (Pin_7), JP30.2 (B); no longer J21.3 (Pin_3)
- net P2r16: now also J21.9 (Pin_9), JP31.2 (B); no longer J21.2 (Pin_2)
- net P2r17: now also J21.10 (Pin_10), JP32.2 (B); no longer J21.1 (Pin_1)
