File: load_switch_12V.kicad_sch (KiCad schematic)
At the start: 20 parts, among them J19 Conn_01x02, J20 Conn_01x03_Odd_Even, J21 Conn_01x02, Q2 AO3401A, Q3 2N7002, Q4 AO3401A, U12 INA199A1DCKR, U13 LMV321-TR, U14 74HC02

Commit message: Rename current limiters to load switches
Parts:
- removed J21: Conn_01x02, HL_Connector_Pad_2.54mm:Pad_1x02_P2.54_1.7x1.7_Rect, symbol Connector_Generic:Conn_01x02
- removed R189: 10k, Resistor_SMD:R_0603_1608Metric_Pad0.98x0.95mm_HandSolder, symbol Device:R_Small
- added D10: RED, LED_SMD:LED_0603_1608Metric, symbol Device:LED
- added D9: GREEN, LED_SMD:LED_0603_1608Metric, symbol Device:LED
- added R10: 2k, Resistor_SMD:R_0603_1608Metric, symbol Device:R
- added R112: 10k, Resistor_SMD:R_0603_1608Metric_Pad0.98x0.95mm_HandSolder, symbol Device:R_Small
- added R9: 1.5k, Resistor_SMD:R_0603_1608Metric, symbol Device:R
- J20: value Conn_01x03_Odd_Even -> Conn_02x03_Odd_Even; footprint HL_Connector_Pad_2.54mm:Pad_1x03_P2.54_1.7x1.7_Rnd-Rnd-Oct -> HL_Connector_Pad_2.54mm:Pad_2x03_P2.54_1.7x1.7_Rect-1Oct-2Rnd; symbol Connector_Generic:Conn_01x03 -> Connector_Generic:Conn_02x03_Odd_Even
Connections:
- net +3.3V: now also R10.1
- net EN: now also R9.1
- net FAULT: now also R112.1
- net FAULT_F: now also R112.2
- net GND: now also J20.1 (Pin_1), J20.3 (Pin_3), J20.5 (Pin_5), D9.1 (K)
- net V_{Iin}: now also J20.2 (Pin_2); no longer J20.3 (Pin_3)
- net Vout: now also J20.4 (Pin_4), J20.6 (Pin_6); no longer J20.1 (Pin_1), J20.2 (Pin_2)
- net ~{LF}: now also D10.1 (K)
- new net: D10.2 (A), R10.2
- new net: D9.2 (A), R9.2

Commit message: Update the design to a stackable one
Parts:
- J15: renamed from J20; value Conn_02x03_Odd_Even -> Conn_02x03_Pin; JLCPCB_CORRECTION 0;2.54;270 -> 1.27;-2.54;270; LCSC C2937625 -> C2685197
- renumbered C67 to C42, C42 to C43, D9 to D17, D10 to D18, J19 to J14, R38 to R36, R39 to R37, R40 to R38, R41 to R39, R112 to R40, R9 to R41, R10 to R42
Connections:
- net V_{Iin} renamed CS
