File: load_switch_5v.kicad_sch (KiCad schematic)
At the start: 10 parts, among them J11 Conn_01x02, J12 Conn_01x04, U4 AP22653AW6-7, U5 INA199A1DCKR

Commit message: Update the design to a stackable one
Parts:
- added D10: RED, LED_SMD:LED_0603_1608Metric, symbol Device:LED
- added D9: GREEN, LED_SMD:LED_0603_1608Metric, symbol Device:LED
- added R21: 1.5k, Resistor_SMD:R_0603_1608Metric, symbol Device:R
- added R22: 2k, Resistor_SMD:R_0603_1608Metric, symbol Device:R
- J7: renamed from J12; value Conn_01x04 -> Conn_02x03_Pin; footprint HL_Connector_Pad_2.54mm:Pad_1x04_P2.54_1.7x1.7_Rect-Rnd-Oct-Rnd -> HL_Connector_Pad_2.54mm:Pad_2x03_P2.54_1.7x1.7_Rect-Rnd-Oct-Rnd; symbol Connector_Generic:Conn_01x04 -> Connector_Generic:Conn_02x03_Odd_Even; JLCPCB_CORRECTION 0;3.81;270 -> 1.27;-2.54;270; LCSC C2691448 -> C2685197
- renumbered J11 to J6, R30 to R20, R31 to R23
Connections:
- net +3.3V: now also R22.1
- net EN: now also R21.1
- net GND: now also J7.3 (Pin_3), J7.5 (Pin_5), D9.1 (K)
- net Vout: now also J7.6 (Pin_6); no longer J7.4 (Pin_4)
- net ~{FAULT}: now also D10.1 (K)
- net V_{Iin} renamed CS
- net CS: now also J7.4 (Pin_4); no longer J7.3 (Pin_3)
- new net: D10.2 (A), R22.2
- new net: D9.2 (A), R21.2
