File: raspi-gpio.kicad_sch (KiCad schematic)
At the start: 3 parts, among them J89 Conn_01x20_RPi_GPIO_Odd, J90 Conn_02x20_Odd_Even, J91 Conn_01x20_RPi_GPIO_Even

Commit message: Rename project to HALSPA
Parts:
- J89: symbol Haltest:Conn_01x20_RPi_GPIO_Odd -> HALSPA:Conn_01x20_RPi_GPIO_Odd
- J91: symbol Haltest:Conn_01x20_RPi_GPIO_Even -> HALSPA:Conn_01x20_RPi_GPIO_Even
Changed lines of the file:
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@@
 	)
 	(symbol
-		(lib_id "Haltest:Conn_01x20_RPi_GPIO_Odd")
+		(lib_id "HALSPA:Conn_01x20_RPi_GPIO_Odd")
 		(at 119.38 83.82 0)
 		(unit 1)
@@
 	)
 	(symbol
-		(lib_id "Haltest:Conn_01x20_RPi_GPIO_Even")
+		(lib_id "HALSPA:Conn_01x20_RPi_GPIO_Even")
 		(at 167.64 83.82 0)
 		(unit 1)
@@
 		)
 		(instances
-			(project "HALTEST"
+			(project "HALSPA"
 				(path "/7eeba806-440e-4671-bc07-69fe183910a7/d60c1020-d2cb-4d48-a4f2-2128439747bd"
 					(reference "#PWR0261")

Commit message: WIP v0.2.0 changes
Parts:
- J77: renamed from J89; symbol HALSPA:Conn_01x20_RPi_GPIO_Odd -> HL_Connector_Pad_2.54mm:Conn_01x20_RPi_GPIO_Odd
- J79: renamed from J91; symbol HALSPA:Conn_01x20_RPi_GPIO_Even -> HL_Connector_Pad_2.54mm:Conn_01x20_RPi_GPIO_Even
- renumbered J90 to J78
Changed lines of the file:
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@@
+			"AAAAAAAAAAAAAAAAAAAAAAAAAAAAAAAAAAAAAAAAAAAAAAAAAAAAAAAAAAAAAAAAAAAAAAAAAAAA"
+			"AAAAAAAAAAAAAAAAAAAAAAAAAAAAAAAAAAAAAAAAAAAAAAAAAAAAAAAAAAAAAAAAAAAAAAAAAAAA"
+			"AAAAAAAAAAAAAAAAAAAAAAAAAAAAAAAAAAAAAAAAAAAAAAAAAAAAAAAAAAAAAAAAAAAAAAAAAAAA"
+			"AAAAAAAAAAAAAAAAAAAAAAAAAAAAAAAAAAAAAAAAAAAAAAAAAAAAAAAAAAAAAAAAAAAAAAAAAAAA"
+			"AAAAAAAAAAAAAAAAAAAAAAAAAAAAAAAAAAAAAAAAAAAAAAAAAAAAAAAAAAAAAAAAAAAAAAAAAAAA"
+			"AAAAAAAAAAAAAAAAAAAAAAAAAAAAAAAAAAAAAAAAAAAAAAAAAAAAAAAAAAAAAAAAAAAAAAAAAAAA"
+			"AAAAAAAAAAAAAAAAAAAAAAAAAAAAAAAAAAAAAAAAAAAAAAAAAAAAAAAAAAAAAAAAAAAAAAAAAAAA"
+			"AAAAAAAAAAAAAAAAAAAAAAAAAAAAAAAAAAAAAAAAAAAAAAAAAAAAAAAAAAAAAAAAAAAAAAAAAAAA"
+			"AAAAAAAAAAAAAAAAAAAAAAAAAAAAAAAAAAAAAAAAAAAAAAAAAAAAAAAAAAAAAAAAAAAAAAAAAAAA"
+			"AAAAAAAAAAAAAAAAAAAAAAAAAAAAAAAAAAAAAAAAAAAAAAAAAAAAAAAAAAAAAAAAAAAAAAAAAAAA"
+			"AAAAAAAAAAAAAAAAAAAAAAAAAAAAAAAAAAAAAAAAAAAAAAAAAAAAAAAAAAAAAAAAAAAAAAAAAAAA"
+			"AAAAAAAAAAAAAAAAAAAAAAAAAAAAAAAAAAAAAAAAAAAAAAAAAAAAAAAAAAAAAAAAAAAAAAAAAAAA"
+			"AAAAAAAAAAAAAAAAAAAAAAAAAAAAAAAAAAAAAAAAAAAAAAAAAAAAAAAAAAAAAAAAAAAAAAAAAAAA"
+			"AAAAAAAAAAAAAAAAAAAAAAAAAAAAAAAAAAAAAAAAAAAAAAAAAAAAAAAAAAAAAAAAAAAAAAAAAAAA"
+			"AAAAAAAAAAAAAAAAAAAAAAAAAAAAAAAAAAAAAAAAAAAAAAAAAAAAAAAAAAAAAAAAAAAAAAAAAAAA"
+			"AAAAAAAAAAAAAAAAAAAAAAAAAAAAAAAAAAAAAAAAAAAAAAAAAAAAAAAAAAAAAAAAAAAAAAAAAAAA"
+			"AAAAAAAAAAAAAAAAAAAAAAAAAAAAAAAAAAAAAAAAAAAAAAAAAAAAAAAAAAAAAAAAAAAAAAAAAAAA"
+			"AAAAAAAAAAAAAAAAAAAAAAAAAAAAAAAAAAAAAAAAAAAAAAAAAAAAAAAAAAAAAAAAAAAAAAAAAAAA"
+			"AAAAAAAAAAAAAAAAAAAAAAAAAAAAAAAAAAAAAAAAAAAAAAAAAAAAAAAAAAAAAAAAAAAAAAAAAAAA"
+			"AAAAAAAAAAAAAAAAAAAAAAAAAAAAAAAAAAAAAAAAAAAAAAAAAAAAAAAAAAAAAAAAAAAAAAAAAAAA"
+			"AAAAAGkAAABaAAAAbwAAADQAAABaAAAAWgAAACsAAAArAAAANgAAAGQAAAByAAAAVgAAADMAAAA3"
+			"AAAAYgAAAGUAAABtAAAATwAAAGEAAABqAAAAMgAAAG8AAABxAAAARgAAADcAAABrAAAAWgAAAFoA"
+			"AAA1AAAAZQAAAGEAAABzAAAAdAAAAEgAAAB5AAAAMgAAAHoAAABWAAAAWQAAAHkAAAA5AAAAYgAA"
+			"ADgAAABkAAAASwAAAFYAAABWAAAAbAAAAE4AAABSAAAAYgAAAHAAAABuAAAASAAAAGoAAAA3AAAA"
+			"SwAAAGMAAABVAAAANAAAADYAAAB6AAAANwAAAGoAAAA2AAAAeQAAAE0AAABEAAAAWgAAACsAAABt"
+			"AAAALwAAAFYAAABlAAAANwAAAEIAAABaAAAAdgAAAFIAAABRAAAAQQAAAEIAAABCAAAASQAAAEwA"
+			"AABBAAAALwAAAGcAAAB3AAAAVQAAAHEAAAByAAAAUAAAAFIAAAB1AAAAbgAAAFcAAAA1AAAAMwAA"
+			"AGwAAABDAAAANAAAAHgAAABGAAAAWgAAACsAAABQAAAASwAAAEoAAABkAAAAMwAAADgAAABIAAAA"
+			"cQAAAGgAAABYAAAALwAAAGYAAAB2AAAAYgAAADgAAABNAAAASwAAAGIAAABwAAAAMAAAAC8AAABk"
+			"AAAANwAAAGIAAAA3AAAAKwAAAEIAAAA5AAAARgAAAFMAAABqAAAAVQAAAE4AAABWAAAAYwAAAGoA"
+			"AABMAAAAVwAAADYAAAA1AAAANQAAAGQAAABZAAAAdwAAAHUAAABrAAAAVAAAADMAAABIAAAARwAA"
+			"AHAAAABzAAAAVgAAAEkAAABOAAAAbAAAAGYAAAAyAAAAOAAAAGsAAAA3AAAATgAAAFcAAAByAAAA"
+			"WgAAADQAAABOAAAAcgAAAGEAAABGAAAATQAAAGYAAABNAAAAVgAAADMAAAByAAAATgAAAGUAAAAv"
+			"AAAAVwAAAEEAAABtAAAAKwAAAEkAAAAvAAAAZgAAAEQAAABEAAAANgAAAFEAAAAwAAAAVwAAAHUA"
+			"AABmAAAAbgAAAG0AAAByAAAANAAAAFoAAAByAAAAbQAAAFUAAABhAAAAcgAAADYAAABIAAAAcgAA"
+			"AFUAAABYAAAARgAAAEgAAABEAAAAdQAAAGYAAABaAAAASAAAAG8AAAB4AAAAdAAAAGYAAABmAAAA"
+			"UAAAAEgAAABGAAAAcwAAAEwAAABoAAAARwAAAFoAAABhAAAAZwAAAGoAAABqAAAASwAAADcAAAA3"
+			"AAAAYQAAAHYAAABpAAAATgAAAGkAAAB1AAAANAAAAG4AAABHAAAAZwAAAGMAAABLAAAAZAAAAGUA"
+			"AAAAAAAAAAAAAAAAAAAAAAAAAAAAAAAAAAAAAAAAAAAAAAAAAAAAAAAAAAAAAAAAAAAAAAAAAAAA"
+			"AAAAAAAAAAAAAAAAAAAAAAAAAAAAAAAAAAAAAAAAAAAAAAAAAAAAAAAAAAAAAAAAAAAAAAAAAAAA"
+			"AAAAAAAAAAAAAAAAAAAAAAAAAAAAAAAAAAAAAAAAAAAAAAAAAAAAAAAAAAAAAAAAAAAAAAAAAAAA"
+			"AAAAAAAAAAAAAAAAAAAAAAAAAAAAAAAAAAAAAAAAAAAAAAAAAAAAAAAAAAAAAAAAAAAAAAAAAAAA"
+			"AAAAAAAAAAAAAAAAAAAAAAAAAAAAAAAAAAAAAAAAAAAAAAAAAAAAAAAAAAAAAAAAAAAAAAAAAAAA"
+			"AAAAAAAAAAAAAAAAAAAAAAAAAAAAAAAAAAAAAAAAAAAAAAAAAAAAAAAAAAAAAAAAAAAAAAAAAAAA"
+			"AAAAAAAAAAAAAAAAAAAAAAAAAAAAAAAAAAAAAAAAAAAAAAAAAAAAAAAAAAAAAAAAAAAAAAAAAAAA"
+			"AAAAAAAAAAAAAAAAAAAAAAAAAAAAAAAAAAAAAAAAAAAAAAAAAAAAAAAAAAAAAAAAAAAAAAAAAAAA"
+			"AAAAAAAAAAAAAAAAAAAAAAAAAAAAAAAAAAAAAAAAAAAAAAAAAAAAAAAAAAAAAAAAAAAAAAAAAAAA"
+			"AAAAAAAAAAAAAAAAAAAAAAAAAAAAAAAAAAAAAAAAAAAAAAAAAAAAAAAAAAAAAAAAAAAAAAAAAAAA"
+			"AAAAAAAAAAAAAAAAAAAAAAAAAAAAAAAAAAAAAAAAAAAAAAAAAAAAAAAAAAAAAAAAAAAAAAAAAAAA"
+			"AAAAAAAAAAAAAAAAAAAAAAAAAAAAAAAAAAAAAAAAAAAAAAAAAAAAAAAAAAAAAAAAAAAAAAAAAAAA"
+			"AAAAAAAAAAAAAAAAAAAAAAAAAAAAAAAAAAAAAAAAAAAAAAAAAAAAAAAAAAAAAAAAAAAAAAAAAAAA"
+			"AAAAAAAAAAAAAAAAAAAAAAAAAAAAAAAAAAAAAAAAAAAAAAAAAAAAAAAAAAAAAAAAAAAAAAAAAAAA"
+			"AAAAAAAAAAAAAAAAAAAAAAAAAAAAAAAAAAAAAAAAAAAAAAAAAAAAAAAAAAAAAAAAAAAAAAAAAAAA"
+			"AAAAAAAAAAAAAAAAAAAAAAAAAAAAAAAAAAAAAAAAAAAAAAAAAAAAAAAAAAAAAAAAAAAAAAAAAAAA"
+			"AAAAAAAAAAAAAAAAAAAAAAAAAAAAAAAAAAAAAAAAAAAAAAAAAAAAAAAAAAAAAAAAAAAAAAAAAAAA"
+			"AAAAAAAAAAAAAAAAAAAAAAAAAAAAAAAAAAAAAAAAAAAAAAAAAAAAAAAAAAAAAAAAAAAAAAAAAAAA"
+			"AP//////////////////////////////////////////////////////////////////////////"
+			"////////////////////////////////////////////////////////////////////////////"
+			"////////////////////////////////////////////////////////////////////////////"
+			"////////////////////////////////////////////////////////////////////////////"
+			"////////////////////////////////////////////////////////////////////////////"
+			"////////////////////////////////////////////////////////////////////////////"
+			"////////////////////////////////////////////////////////////////////////////"
+			"////////////////////////////////////////////////////////////////////////////"
+			"////////////////////////////////////////////////////////////////////////////"
+			"////////////////////////////////////////////////////////////////////////////"
+			"////////////////////////////////////////////////////////////////////////////"
+			"////////////////////////////////////////////////////////////////////////////"
+			"////////////////////////////////////////////////////////////////////////////"
+			"////////////////////////////////////////////////////////////////////////////"
+			"////////////////////////////////////////////////////////////////////////////"
+			"////////////////////////////////////////////////////////////////////////////"
+			"////////////////////////////////////////////////////////////////////////////"
+			"////////////////////////////////////////////////////////////////////////////"
+			"/wAAAAAAAAAAAAAAAAAAAAAAAAAAAAAAAAAAAAAAAAAAAAAAAAAAAAAAAAAAAAAAAAAAAAAAAAAA"
+			"AAAAAAAAAAAAAAAAAAAAAAAAAAAAAAAAAAAAAAAAAAAAAAAAAAAAAAAAAAAAAAAAAAAAAAAAAAAA"
+			"AAAAAAAAAAAAAAAAAAAAAAAAAAAAAAAAAAAAAAAAAAAAAAAAAAAAAAAAAAAAAAAAAAAAAAAAAAAA"
+			"AAAAAAAAAAAAAAAAAAAAAAAAAAAAAAAAAAAAAAAAAAAAAAAAAAAAAAAAAAAAAAAAAAAAAAAAAAAA"
+			"AAAAAAAAAAAAAAAAAAAAAAAAAAAAAAAAAAAAAAAAAAAAAAAAAAAAAAAAAAAAAAAAAAAAAAAAAAAA"
+			"AAAAAAAAAAAAAAAAAAAAAAAAAAAAAAAAAAAAAAAAAAAAAAAAAAAAAAAAAAAAAAAAAAAAAAAAAAAA"
+			"AAAAAAAAAAAAAAAAAAAAAAAAAAAAAAAAAAAAAAAAAAAAAAAAAAAAAAAAAAAAAAAAAAAAAAAAAAAA"
+			"AAAAAAAAAAAAAAAAAAAAAAAAAAAAAAAAAAAAAAAAAAAAAAAAAAAAAAAAAAAAAAAAAAAAAAAAAAAA"
+			"AAAAAAAAAAAAAAAAAAAAAAAAAAAAAAAAAAAAAAAAAAAAAAAAAAAAAAAAAAAAAAAAAAAAAAAAAAAA"
+			"AAAAAAAAAAAAAAAAAAAAAAAAAAAAAAAAAAAAAAAAAAAAAAAAAAAAAAAAAAAAAAAAAAAAAAAAAAAA"
+			"AAAAAAAAAAAAAAAAAAAAAAAAAAAAAAAAAAAAAAAAAAAAAAAAAAAAAAAAAAAAAAAAAAAAAAAAAAAA"
+			"AAAAAAAAAAAAAAAAAAAAAAAAAAAAAAAAAAAAAAAAAAAAAAAAAAAAAAAAAAAAAAAAAAAAAAAAAAAA"
+			"AAAAAAAAAAAAAAAAAAAAAAAAAAAAAAAAAAAAAAAAAAAAAAAAAAAAAAAAAAAAAAAAAAAAAAAAAAAA"
+			"AAAAAAAAAAAAAAAAAAAAAAAAAAAAAAAAAAAAAAAAAAAAAAAAAAAAAAAAAAAAAAAAAAAAAAAAAAAA"
+			"AAAAAAAAAAAAAAAAAAAAAAAAAAAAAAAAAAAAAAAAAAAAAAAAAAAAAAAAAAAAAAAAAAAAAAAAAAAA"
+			"AAAAAAAAAAAAAAAAAAAAAAAAAAAAAAAAAAAAAAAAAAAAAAAAAAAAAAAAAAAAAAAAAAAAAAAAAAAA"
 			"AAAAAAAAAAAAAAAAAAAAAAAAAAAAAAAAAAAAAAAAAAAAAAAAAAAAAAAAAAAAAAAAAAAAAAAAAAAA"
 			"AAAAAAAAAAAAAAAAAAAAAAAAAAAAAAAAAAAAAAAAAAAAAAAAAAAAAAAAAAAAAAAAAAAAAAAAAAAA"
@@
 	)
 	(symbol
-		(lib_id "HALSPA:Conn_01x20_RPi_GPIO_Odd")
+		(lib_id "HL_Connector_Pad_2.54mm:Conn_01x20_RPi_GPIO_Odd")
 		(at 119.38 83.82 0)
 		(unit 1)
@@
 		(dnp no)
 		(fields_autoplaced yes)
-		(property "Reference" "J89"
+		(property "Reference" "J77"
 			(at 119.38 54.61 0)
 			(effects
@@
 			(project ""
 				(path "/7eeba806-440e-4671-bc07-69fe183910a7/d60c1020-d2cb-4d48-a4f2-2128439747bd"
-					(reference "J89")
+					(reference "J77")
 					(unit 1)
 				)
@@
 		(dnp no)
 		(fields_autoplaced yes)
-		(property "Reference" "J90"
+		(property "Reference" "J78"
 			(at 143.51 54.61 0)
 			(effects
@@
 			(project ""
 				(path "/7eeba806-440e-4671-bc07-69fe183910a7/d60c1020-d2cb-4d48-a4f2-2128439747bd"
-					(reference "J90")
+					(reference "J78")
 					(unit 1)
 				)
@@
 	)
 	(symbol
-		(lib_id "HALSPA:Conn_01x20_RPi_GPIO_Even")
+		(lib_id "HL_Connector_Pad_2.54mm:Conn_01x20_RPi_GPIO_Even")
 		(at 167.64 83.82 0)
 		(unit 1)
@@
 		(dnp no)
 		(fields_autoplaced yes)
-		(property "Reference" "J91"
+		(property "Reference" "J79"
 			(at 170.18 83.8199 0)
 			(effects
@@
 			(project ""
 				(path "/7eeba806-440e-4671-bc07-69fe183910a7/d60c1020-d2cb-4d48-a4f2-2128439747bd"
-					(reference "J91")
+					(reference "J79")
 					(unit 1)
 				)
@@
 		(dnp no)
 		(fields_autoplaced yes)
-		(property "Reference" "#PWR0260"
+		(property "Reference" "#PWR0261"
 			(at 135.89 118.11 0)
 			(effects
@@
 			(project ""
 				(path "/7eeba806-440e-4671-bc07-69fe183910a7/d60c1020-d2cb-4d48-a4f2-2128439747bd"
-					(reference "#PWR0260")
+					(reference "#PWR0261")
 					(unit 1)
 				)
@@
 		(dnp no)
 		(fields_autoplaced yes)
-		(property "Reference" "#PWR0261"
+		(property "Reference" "#PWR0262"
 			(at 151.13 118.11 0)
 			(effects
@@
 			(project "HALSPA"
 				(path "/7eeba806-440e-4671-bc07-69fe183910a7/d60c1020-d2cb-4d48-a4f2-2128439747bd"
-					(reference "#PWR0261")
+					(reference "#PWR0262")
 					(unit 1)
 				)

Commit message: Assign part numbers and finish other 0.2.0 changes
Parts:
- J88: renamed from J77; LCSC (none) -> C50981
- J89: renamed from J78; LCSC (none) -> C9138; THT_LCSC C9138 -> (none)
- J90: renamed from J79; LCSC (none) -> C50981
Changed lines of the file:
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@@
+			"AAAAAAAAAAAAAAAAAAAAAAAAAAAAAAAAAAAAAAAAAAAAAAAAAAAAAAAAAAAAAAAAAAAAAAAAAAAA"
+			"AAAAAAAAAAAAAAAAAAAAAAAAAAAAAAAAAAAAAAAAAAAAAAAAAAAAAAAAAAAAAAAAAAAAAAAAAAAA"
+			"AICNB9mNBwazwY4Hny4KBkucjwcYRgsGjsiPB0vpDAb0CpAHTukMBvQKkAe1rA8G9AqQBwkKEQaf"
+			"048HYWcSBkucjwcnCBUGs8GOB3J+FwaMgI0HvboZBsHgiwfxrhsGjeyJB7xOHQZCsIcHPIodBnw7"
+			"hwfg+B0GWWKGB91CHgYf0YUH448eBvc5hQd7ah8GMZmCByTZHwaC3n8HJNkfBh4bfQck2R8GGht9"
+			"B3tqHwZxYHoHe2ofBm9gegfjjx4Gqb93B4ikHQbA8XUHm0BKBsDxdQebQEoG4weHB4FDSgakI4cH"
+			"/kVKBns7hwdcdkoGP7CHB+/tSgbt0IgHmg5LBjX5iAehDksGPfmIB1lSUQb0PI8HonpRBqFdjwcV"
+			"EFMGkgWQB61DUwb0CpAHzVlkBvUKkAdrjWQGkgWQB90iZgahXY8HLUtmBu88jwfkjmwGN/mIB5Gv"
+			"bAbu0IgHgldtBns7hwfkXG0G4weHB+VcbQbD8XUH5VxtBsDxdQdbxJcGwPF1B1vElwbjB4cHQceX"
+			"BqQjhwe+yZcGezuHBxz6lwY/sIcHr3GYBu3QiAdakpgGNfmIB2GSmAY9+YgHGdaeBvQ8jwdi/p4G"
+			"oV2PB9WToAaSBZAHbcegBvQKkAeN3bEG9QqQBysRsgaSBZAHnaazBqFdjwftzrMG7zyPB6QSugY3"
+			"+YgHUTO6Bu7QiAdC27oGezuHB6TgugbjB4cHpeC6BsPxdQel4LoGwPF1BzuGvgbA8XUHO4a+BuMH"
+			"hwchib4GpCOHB56LvgZ7O4cH/Lu+Bj+whwePM78G7dCIBzpUvwY1+YgHQVS/Bj35iAf5l8UG9DyP"
+			"B0LAxQahXY8HtVXHBpIFkAdNiccG9AqQB22f2Ab1CpAHC9PYBpIFkAd9aNoGoV2PB82Q2gbvPI8H"
+			"hNTgBjf5iAcx9eAG7tCIByKd4QZ7O4cHhKLhBuMHhweFouEGw/F1B4Wi4QbA8XUHG0jlBsDxdQcb"
+			"SOUG4weHBwFL5QakI4cHfk3lBns7hwfcfeUGP7CHB2/15Qbt0IgHGhbmBjX5iAchFuYGPfmIB9lZ"
+			"7Ab0PI8HIoLsBqFdjweVF+4GkgWQBy1L7gb0CpAHTWH/BvUKkAfrlP8GkgWQB10qAQehXY8HrVIB"
+			"B+88jwdklgcHN/mIBxG3Bwfu0IgHAl8IB3s7hwdkZAgH4weHB2VkCAfD8XUHZWQIB8DxdQf7CQwH"
+			"wPF1B/sJDAfjB4cH4QwMB6QjhwdeDwwHezuHB7w/DAc/sIcHT7cMB+3QiAf61wwHNfmIBwHYDAc9"
+			"+YgHuRsTB/Q8jwcCRBMHoV2PB3XZFAeSBZAHDQ0VB/QKkActIyYH9QqQB8tWJgeSBZAHPewnB6Fd"
+			"j465HIE5rw1xSz+XXqGbN0kFirqu0knHucodW0sViioHkYRppyn3IapSLP9xgpvz7Ltuz+bNrnCZ"
+			"sq7qaZ1cJdmv3FEN0jbN7hfREIUEbUICbJAH2eaRhHsRgYNkHxE8GCyhiEIydTpIuWZKKIYraQgp"
+			"M03utQR5LJJsn71yz/T3U+79BGdQGhQbJNAG5PhGFDrNXCNAFozIZI+1UFFgzJgxbuCgp/Qasd4h"
+			"XFsy9Sld3rJFizRbOZrjU1Hg66+/0b7BY8aO1SHaSPboGUKEseY2btwo4rChiELWTWxW1upwJVFZ"
+			"vwkSRueYLgQhmY2eJOSAZPT1v/027SlMGdRgYS19QwgoKinwHUbatGkjOsJFrptUHkgUQpAyrVQl"
+			"eOmll1WvIUjouGOPlbLjV+q2fNf5Hj/77HO6P78tKjzcd++9kkl5nL73wgsvuo8+/lj1MX6z6BCU"
+			"J6UMeuvWrf6FfSiikLmc1K2bXjPG//LLoarf/PDjj7o/OglzOl4qLzQMOFd6+lF2FL3kjTfeVJ0H"
+			"gvgMIR0JQmsl5eFzA1H47rvvSn/NjzQIiwzS4nIvY/4QnT16nKG6m4Jt/xkChkBUCBhRGBVstpMh"
+			"YAgYAnkXgcwShSiwKKg43pavSI3AC4cOTre2bY9xx0gGwzHHtD1IkQtHFKpzUaJXyaAIJftFKcc4"
+			"wDFJjwGiQDF8MEAxCihPRhkVovpwiHrJT0QhDoF4iRjs3Dm1txO9CjFe4iXKEAoOzHB+TpBMCshC"
+			"en+QEYLESbQxfZzuuusuNSQrVkztsaAfxui/9VNnu2XDfnHrJ85we4XkLXNUE1ftzC6uapc2EY+w"
+			"U4jClb9MTCUKJ03V3jREh1eSrMIjCh6cgRhxIPvQEDAEDIEICMwTx9Nngz91W7amlocO3rQkRF7l"
+			"aq54ieKusGTLZ0U27djm/lmz3M2Sx6KNa3UoSCwcUjibTjyxa8ThKbNFBiFrHGsjDuOpU6dqphzr"
+			"NdHnHSTynSw6+hGRTRLssPUHiJYo5DjPSI/CESO+1Yh+iEIcORCErMu1atX0hwj5zLw3bdrs5iUl"
+			"SbnQvw/aZqBE699ww/VpBN5BHx74A2chGQ1kFuAsJKAJB+kUyXLBicn4zIMofgKRcJaHc3wHjk8Q"
+			"0ldffaUOUAhHMKYHYs+ePTWSHSdmoHwh2wwbNkxxwJlVuEBBlxBfyrWoXNN1SIxNRuF6WbsXLFqQ"
+			"FhwVeHxeN2rQ2HXq2NlVlJJ/6FMmhkBeQWDd2Clu01+z3H75HZZsWN9V6nasq9KlrStZu2rEU9ww"
+			"Y55bis45YbqUsk92ZdE5e3RyVbvFnpiJOJEIH0ZDFGJHTZgwUXX5+fOTIozuxCaI17Wge/eTlTgJ"
+			"3gAAAAAAAAAAAAAAAAAAAAAAAAAAAAAAAAAAAAAAAAAAAAAAAAAAAAAAAAAAAAAAAAAAAAAAAAAA"
+			"AAAAAAAAAAAAAAAAAAAAAAAAAAAAAAAAAAAAAAAAAAAAAAAAAAAAAAAAAAAAAAAAAAAAAAAAAAAA"
+			"AAAAAAAAAAAAAAAAAAAAAAAAAAAAAAAAAAAAAAAAAAAAAAAAAAAAAAAAAAAAAAAAAAAAAAAAAAAA"
+			"AAAAAAAAAAAAAAAAAAAAAAAAAAAAAAAAAAAAAAAAAAAAAAAAAAAAAAAAAAAAAAAAAAAAAAAAAAAA"
+			"AAAAAAAAAAAAAAAAAAAAAAAAAAAAAAAAAAAAAAAAAAAAAAAAAAAAAAAAAAAAAAAAAAAAAAAAAAAA"
+			"AAAAAAAAAAAAAAAAAAAAAAAAAAAAAAAAAAAAAAAAAAAAAAAAAAAAAAAAAAAAAAAAAAAAAAAAAAAA"
+			"AAAAAAAAAAAAAAAAAAAAAAAAAAAAAAAAAAAAAAAAAAAAAAAAAAAAAAAAAAAAAAAAAAAAAAAAAAAA"
+			"AAAAAAAAAAAAAAAAAAAAAAAAAAAAAAAAAAAAAAAAAAAAAAAAAAAAAAAAAAAAAAAAAAAAAAAAAAAA"
+			"AAAAAAAAAAAAAAAAAAAAAAAAAAAAAAAAAAAAAAAAAAAAAAAAAAAAAAAAAAAAAAAAAAAAAAAAAAAA"
+			"AAAAAAAAAAAAAAAAAAAAAAAAAAAAAAAAAAAAAAAAAAAAAAAAAAAAAAAAAAAAAAAAAAAAAAAAAAAA"
+			"AAAAAAAAAAAAAAAAAAAAAAAAAAAAAAAAAAAAAAAAAAAAAAAAAAAAAAAAAAAAAAAAAAAAAAAAAAAA"
+			"AAAAAAAAAAAAAAAAAAAAAAAAAAAAAAAAAAAAAAAAAAAAAAAAAAAAAAAAAAAAAAAAAAAAAAAAAAAA"
+			"AAAAAAAAAAAAAAAAAAAAAAAAAAAAAAAAAAAAAAAAAAAAAAAAAAAAAAAAAAAAAAAAAAAAAAAAAAAA"
+			"AAAAAAAAAAAAAAAAAAAAAAAAAAAAAAAAAAAAAAAAAAAAAAAAAAAAAAAAAAAAAAAAAAAAAAAAAAAA"
+			"AAAAAAAAAAAAAAAAAAAAAAAAAAAAAAAAAAAAAAAAAAAAAAAAAAAAAAAAAAAAAAAAAAAAAAAAAAAA"
+			"AAAAAAAAAAAAAAAAAAAAAAAAAAAAAAAAAAAAAAAAAAAAAAAAAAAAAAAAAAAAAAAAAAAAAAAAAAAA"
 			"AAAAAAAAAAAAAAAAAAAAAAAAAAAAAAAAAAAAAAAAAAAAAAAAAAAAAAAAAAAAAAAAAAAAAAAAAAAA"
 			"AAAAAAAAAAAAAAAAAAAAAAAAAAAAAAAAAAAAAAAAAAAAAAAAAAAAAAAAAAAAAAAAAAAAAAAAAAAA"
@@
 		(dnp no)
 		(fields_autoplaced yes)
-		(property "Reference" "J77"
+		(property "Reference" "J88"
 			(at 119.38 54.61 0)
 			(effects
@@
 					(size 1.27 1.27)
 				)
+			)
+		)
+		(property "LCSC" "C50981"
+			(at 119.38 83.82 0)
+			(effects
+				(font
+					(size 1.27 1.27)
+				)
+				(hide yes)
 			)
 		)
@@
 			(project ""
 				(path "/7eeba806-440e-4671-bc07-69fe183910a7/d60c1020-d2cb-4d48-a4f2-2128439747bd"
-					(reference "J77")
+					(reference "J88")
 					(unit 1)
 				)
@@
 		(dnp no)
 		(fields_autoplaced yes)
-		(property "Reference" "J78"
+		(property "Reference" "J89"
 			(at 143.51 54.61 0)
 			(effects
@@
 			)
 		)
-		(property "LCSC" ""
+		(property "LCSC" "C9138"
 			(at 142.24 83.82 0)
 			(effects
@@
 			)
 		)
-		(property "THT_LCSC" "C9138"
+		(property "THT_LCSC" ""
 			(at 142.24 83.82 0)
 			(effects
@@
 			(project ""
 				(path "/7eeba806-440e-4671-bc07-69fe183910a7/d60c1020-d2cb-4d48-a4f2-2128439747bd"
-					(reference "J78")
+					(reference "J89")
 					(unit 1)
 				)
@@
 		(dnp no)
 		(fields_autoplaced yes)
-		(property "Reference" "J79"
+		(property "Reference" "J90"
 			(at 170.18 83.8199 0)
 			(effects
@@
 					(size 1.27 1.27)
 				)
+			)
+		)
+		(property "LCSC" "C50981"
+			(at 167.64 83.82 0)
+			(effects
+				(font
+					(size 1.27 1.27)
+				)
+				(hide yes)
 			)
 		)
@@
 			(project ""
 				(path "/7eeba806-440e-4671-bc07-69fe183910a7/d60c1020-d2cb-4d48-a4f2-2128439747bd"
-					(reference "J79")
+					(reference "J90")
 					(unit 1)
 				)
@@
 		(dnp no)
 		(fields_autoplaced yes)
-		(property "Reference" "#PWR0261"
+		(property "Reference" "#PWR0270"
 			(at 135.89 118.11 0)
 			(effects
@@
 			(project ""
 				(path "/7eeba806-440e-4671-bc07-69fe183910a7/d60c1020-d2cb-4d48-a4f2-2128439747bd"
-					(reference "#PWR0261")
+					(reference "#PWR0270")
 					(unit 1)
 				)
@@
 		(dnp no)
 		(fields_autoplaced yes)
-		(property "Reference" "#PWR0262"
+		(property "Reference" "#PWR0271"
 			(at 151.13 118.11 0)
 			(effects
@@
 			(project "HALSPA"
 				(path "/7eeba806-440e-4671-bc07-69fe183910a7/d60c1020-d2cb-4d48-a4f2-2128439747bd"
-					(reference "#PWR0262")
+					(reference "#PWR0271")
 					(unit 1)
 				)

Commit message: Update the title blocks
Other:
- company: (none) -> Hat Labs Oy
- title: (none) -> HALSPA - Hat Labs Spaghetti Board
Changed lines of the file:
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@@
 	(generator_version "9.0")
 	(paper "A4")
+	(title_block
+		(title "HALSPA - Hat Labs Spaghetti Board")
+		(date "2025-04-17")
+		(rev "v0.2.0")
+		(company "Hat Labs Oy")
+		(comment 1 "See the accompanying LICENSE.md file for license details.")
+	)
 	(junction
 		(at 151.13 66.04)
@@
 			"AAAAAAAAAAAAAAAAAAAAAAAAAAAAAAAAAAAAAAAAAAAAAAAAAAAAAAAAAAAAAAAAAAAAAAAAAAAA"
 			"AAAAAAAAAAAAAAAAAAAAAAAAAAAAAAAAAAAAAAAAAAAAAAAAAAAAAAAAAAAAAAAAAAAAAAAAAAAA"
+			"AAAAAAAAAAAAAAAAAAAAAAAAAAAAAAAAAAAAAAAAAAAAAAAAAAAAAAAAAAAAAAAAAAAAAAAAAAAA"
+			"AAAAAAAAAAAAAAAAAAAAAAAAAAAAAAAAAAAAAAAAAAAAAAAAAAAAAAAAAAAAAAAAAAAAAAAAAAAA"
+			"AAAAAAAAAAAAAAAAAAAAAAAAAAAAAAAAAAAAAAAAAAAAAAAAAAAAAAAAAAAAAAAAAAAAAAAAAAAA"
+			"AAAAAAAAAAAAAAAAAAAAAAAAAAAAAAAAAAAAAAAAAAAAAAAAAAAAAAAAAAAAAAAAAAAAAAAAAAAA"
+			"AAAAAAAAAAAAAAAAAAAAAAAAAAAAAAAAAAAAAAAAAAAAAAAAAAAAAAAAAAAAAAAAAAAAAAAAAAAA"
+			"AAAAAAAAAAAAAAAAAAAAAAAAAAAAAAAAAAAAAAAAAAAAAAAAAAAAAAAAAAAAAAAAAAAAAAAAAAAA"
+			"AAAAAAAAAAAAAAAAAAAAAAAAAAAAAAAAAAAAAAAAAAAAAAAAAAAAAAAAAAAAAAAAAAAAAAAAAAAA"
+			"AAAAAAAAAAAAAAAAAAAAAAAAAAAAAAAAAAAAAAAAAAAAAAAAAAAAAAAAAAAAAAAAAAAAAAAAAAAA"
+			"AAAAAAAAAAAAAAAAAAAAAAAAAAAAAAAAAAAAAAAAAAAAAAAAAAAAAAAAAAAAAAAAAAAAAAAAAAAA"
+			"AAAAAAAAAAAAAAAAAAAAAAAAAAAAAAAAAAAAAAAAAAAAAAAAAAAAAAAAAAAAAAAAAAAAAAAAAAAA"
+			"AAAAAAAAAAAAAAAAAAAAAAAAAAAAAAAAAAAAAAAAAAAAAAAAAAAAAAAAAAAAAAAAAAAAAAAAAAAA"
+			"AAAAAAAAAAAAAAAAAAAAAAAAAAAAAAAAAAAAAAAAAAAAAAAAAAAAAAAAAAAAAAAAAAAAAAAAAAAA"
+			"AAAAAAAAAAAAAAAAAAAAAAAAAAAAAAAAAAAAAAAAAAAAAAAAAAAAAAAAAAAAAAAAAAAAAAAAAAAA"
+			"AAAAAAAAAAAAAAAAAAAAAAAAAAAAAAAAAAAAAAAAAAAAAAAAAAAAAAAAAAAAAAAAAAAAAAAAAAAA"
+			"AAAAAAAAAAAAAAAAAAAAAAAAAAAAAAAAAAAAAAAAAAAAAAAAAAAAAAAAAAAAAAAAAAAAAAAAAAAA"
+			"AAAAAAAAAAAAAAAAAAAAAAAAAAAAAAAAAAAAAAAAAAAAAAAAAAAAAAAAAAAAAAAAAAAAAAAAAAAA"
+			"AAAAAAAAAAAAAAAAAAAAAAAAAAAAAAAAAAAAAAAAAAAAAAAAAAAAAAAAAAAAAAAAAAAAAAAAAAAA"
+			"AAAAAAAAAAAAAAAAAAAAAAAAAAAAAAAAAAAAAAAAAAAAAAAAAAAAAAAAAAAAAAAAAAAAAAAAAAAA"
