File: usb_serial.kicad_sch (KiCad schematic)
At the start: 13 parts, among them J53 USB_B_Micro, J54 Conn_02x04_Odd_Even, Q8 S8050, Q9 S8050, U27 CH340C

Commit message: Replace micro-usb connectors with horizontal ones
Parts:
- J53: footprint HL_Connector_USB:MICRO-USB-SMD_MICRO-21-P2-T3 -> HL_Connector_USB:MICRO-USB-SMD_MICROXNJ; LCSC C2834965 -> C404969
Changed lines of the file:
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@@
 			)
 		)
-		(property "Footprint" "HL_Connector_USB:MICRO-USB-SMD_MICRO-21-P2-T3"
+		(property "Footprint" "HL_Connector_USB:MICRO-USB-SMD_MICROXNJ"
 			(at 57.15 77.47 0)
 			(effects
@@
 			)
 		)
-		(property "LCSC" "C2834965"
+		(property "LCSC" "C404969"
 			(at 53.34 76.2 0)
 			(effects

Commit message: Update the design to a stackable one
Parts:
- J37: renamed from J53; footprint HL_Connector_USB:MICRO-USB-SMD_MICROXNJ -> HL_Connector_USB:MICRO-USB-SMD_920-154A2021Y10109; LCSC C404969 -> C399946
- J38: renamed from J54; value Conn_02x04_Odd_Even -> Conn_02x04_Pin; JLCPCB_CORRECTION 1.27;3.81;270 -> 1.27;-3.81;270
- renumbered C56 to C66, C57 to C67, JP1 to JP33, JP2 to JP34, R104 to R108, R105 to R109, R106 to R110, R107 to R111
Changed lines of the file:
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@@
 	(title_block
 		(title "HALSPA - Hat Labs Spaghetti Board")
-		(date "2025-08-15")
-		(rev "v0.3.0")
+		(date "2025-10-17")
+		(rev "v0.4.0")
 		(company "Hat Labs Oy")
 		(comment 1 "https://ohwr.org/cern_ohl_s_v2.pdf")
@@
 		(on_board yes)
 		(dnp no)
-		(property "Reference" "J53"
+		(property "Reference" "J37"
 			(at 54.7878 64.3382 0)
 			(effects
@@
 			)
 		)
-		(property "Footprint" "HL_Connector_USB:MICRO-USB-SMD_MICROXNJ"
+		(property "Footprint" "HL_Connector_USB:MICRO-USB-SMD_920-154A2021Y10109"
 			(at 57.15 77.47 0)
 			(effects
@@
 			)
 		)
-		(property "LCSC" "C404969"
+		(property "LCSC" "C399946"
 			(at 53.34 76.2 0)
 			(effects
@@
 			(project "HALSPA"
 				(path "/7eeba806-440e-4671-bc07-69fe183910a7/d2563b9c-21b7-43a8-ad57-d0568fac8495"
-					(reference "J53")
+					(reference "J37")
 					(unit 1)
 				)
@@
 		(on_board yes)
 		(dnp no)
-		(property "Reference" "R105"
+		(property "Reference" "R109"
 			(at 149.86 83.6422 90)
 			(effects
@@
 			(project "HALSPA"
 				(path "/7eeba806-440e-4671-bc07-69fe183910a7/d2563b9c-21b7-43a8-ad57-d0568fac8495"
-					(reference "R105")
+					(reference "R109")
 					(unit 1)
 				)
@@
 		(on_board yes)
 		(dnp no)
-		(property "Reference" "#PWR0216"
+		(property "Reference" "#PWR0226"
 			(at 190.5 72.39 0)
 			(effects
@@
 			(project "HALSPA"
 				(path "/7eeba806-440e-4671-bc07-69fe183910a7/d2563b9c-21b7-43a8-ad57-d0568fac8495"
-					(reference "#PWR0216")
+					(reference "#PWR0226")
 					(unit 1)
 				)
@@
 		(on_board yes)
 		(dnp no)
-		(property "Reference" "R106"
+		(property "Reference" "R110"
 			(at 188.468 92.8116 0)
 			(effects
@@
 			(project "HALSPA"
 				(path "/7eeba806-440e-4671-bc07-69fe183910a7/d2563b9c-21b7-43a8-ad57-d0568fac8495"
-					(reference "R106")
+					(reference "R110")
 					(unit 1)
 				)
@@
 		(on_board yes)
 		(dnp no)
-		(property "Reference" "C57"
+		(property "Reference" "C67"
 			(at 193.421 61.0616 0)
 			(effects
@@
 			(project "HALSPA"
 				(path "/7eeba806-440e-4671-bc07-69fe183910a7/d2563b9c-21b7-43a8-ad57-d0568fac8495"
-					(reference "C57")
+					(reference "C67")
 					(unit 1)
 				)
@@
 		(dnp no)
 		(fields_autoplaced yes)
-		(property "Reference" "J54"
+		(property "Reference" "J38"
 			(at 240.03 68.58 0)
 			(effects
@@
 			)
 		)
-		(property "Value" "Conn_02x04_Odd_Even"
+		(property "Value" "Conn_02x04_Pin"
 			(at 240.03 71.12 0)
 			(effects
@@
 			)
 		)
-		(property "JLCPCB_CORRECTION" "1.27;3.81;270"
+		(property "JLCPCB_CORRECTION" "1.27;-3.81;270"
 			(at 238.76 77.47 0)
 			(effects
@@
 			(project ""
 				(path "/7eeba806-440e-4671-bc07-69fe183910a7/d2563b9c-21b7-43a8-ad57-d0568fac8495"
-					(reference "J54")
+					(reference "J38")
 					(unit 1)
 				)
@@
 		(on_board yes)
 		(dnp no)
-		(property "Reference" "JP2"
+		(property "Reference" "JP34"
 			(at 115.5699 91.44 90)
 			(effects
@@
 			(project "HALSPA"
 				(path "/7eeba806-440e-4671-bc07-69fe183910a7/d2563b9c-21b7-43a8-ad57-d0568fac8495"
-					(reference "JP2")
+					(reference "JP34")
 					(unit 1)
 				)
@@
 		(on_board yes)
 		(dnp no)
-		(property "Reference" "#PWR0217"
+		(property "Reference" "#PWR0227"
 			(at 229.87 74.93 0)
 			(effects
@@
 			(project "HALSPA"
 				(path "/7eeba806-440e-4671-bc07-69fe183910a7/d2563b9c-21b7-43a8-ad57-d0568fac8495"
-					(reference "#PWR0217")
+					(reference "#PWR0227")
 					(unit 1)
 				)
@@
 		(on_board yes)
 		(dnp no)
-		(property "Reference" "R107"
+		(property "Reference" "R111"
 			(at 192.278 52.1716 0)
 			(effects
@@
 			(project "HALSPA"
 				(path "/7eeba806-440e-4671-bc07-69fe183910a7/d2563b9c-21b7-43a8-ad57-d0568fac8495"
-					(reference "R107")
+					(reference "R111")
 					(unit 1)
 				)
@@
 		(on_board yes)
 		(dnp no)
-		(property "Reference" "R104"
+		(property "Reference" "R108"
 			(at 149.86 64.5922 90)
 			(effects
@@
 			(project "HALSPA"
 				(path "/7eeba806-440e-4671-bc07-69fe183910a7/d2563b9c-21b7-43a8-ad57-d0568fac8495"
-					(reference "R104")
+					(reference "R108")
 					(unit 1)
 				)
@@
 		(on_board yes)
 		(dnp no)
-		(property "Reference" "#PWR0213"
+		(property "Reference" "#PWR0223"
 			(at 105.41 60.96 0)
 			(effects
@@
 			(project "HALSPA"
 				(path "/7eeba806-440e-4671-bc07-69fe183910a7/d2563b9c-21b7-43a8-ad57-d0568fac8495"
-					(reference "#PWR0213")
+					(reference "#PWR0223")
 					(unit 1)
 				)
@@
 		(dnp no)
 		(fields_autoplaced yes)
-		(property "Reference" "#PWR0215"
+		(property "Reference" "#PWR0225"
 			(at 190.5 52.07 0)
 			(effects
@@
 			(project "HALSPA"
 				(path "/7eeba806-440e-4671-bc07-69fe183910a7/d2563b9c-21b7-43a8-ad57-d0568fac8495"
-					(reference "#PWR0215")
+					(reference "#PWR0225")
 					(unit 1)
 				)
@@
 		(on_board yes)
 		(dnp no)
-		(property "Reference" "JP1"
+		(property "Reference" "JP33"
 			(at 118.1101 83.82 90)
 			(effects
@@
 			(project "HALSPA"
 				(path "/7eeba806-440e-4671-bc07-69fe183910a7/d2563b9c-21b7-43a8-ad57-d0568fac8495"
-					(reference "JP1")
+					(reference "JP33")
 					(unit 1)
 				)
@@
 		(on_board yes)
 		(dnp no)
-		(property "Reference" "#PWR0212"
+		(property "Reference" "#PWR0222"
 			(at 93.98 100.33 0)
 			(effects
@@
 			(project "HALSPA"
 				(path "/7eeba806-440e-4671-bc07-69fe183910a7/d2563b9c-21b7-43a8-ad57-d0568fac8495"
-					(reference "#PWR0212")
+					(reference "#PWR0222")
 					(unit 1)
 				)
@@
 		(on_board yes)
 		(dnp no)
-		(property "Reference" "#PWR0210"
+		(property "Reference" "#PWR0220"
 			(at 53.34 99.06 0)
 			(effects
@@
 			(project "HALSPA"
 				(path "/7eeba806-440e-4671-bc07-69fe183910a7/d2563b9c-21b7-43a8-ad57-d0568fac8495"
-					(reference "#PWR0210")
+					(reference "#PWR0220")
 					(unit 1)
 				)
@@
 		(on_board yes)
 		(dnp no)
-		(property "Reference" "#PWR0218"
+		(property "Reference" "#PWR0228"
 			(at 246.38 88.9 0)
 			(effects
@@
 			(project "HALSPA"
 				(path "/7eeba806-440e-4671-bc07-69fe183910a7/d2563b9c-21b7-43a8-ad57-d0568fac8495"
-					(reference "#PWR0218")
+					(reference "#PWR0228")
 					(unit 1)
 				)
@@
 		(dnp no)
 		(fields_autoplaced yes)
-		(property "Reference" "C56"
+		(property "Reference" "C66"
 			(at 99.06 46.99 90)
 			(effects
@@
 			(project "HALSPA"
 				(path "/7eeba806-440e-4671-bc07-69fe183910a7/d2563b9c-21b7-43a8-ad57-d0568fac8495"
-					(reference "C56")
+					(reference "C66")
 					(unit 1)
 				)
@@
 		(dnp no)
 		(fields_autoplaced yes)
-		(property "Reference" "#PWR0214"
+		(property "Reference" "#PWR0224"
 			(at 186.69 92.71 0)
 			(effects
@@
 			(project "HALSPA"
 				(path "/7eeba806-440e-4671-bc07-69fe183910a7/d2563b9c-21b7-43a8-ad57-d0568fac8495"
-					(reference "#PWR0214")
+					(reference "#PWR0224")
 					(unit 1)
 				)
@@
 		(dnp no)
 		(fields_autoplaced yes)
-		(property "Reference" "#PWR0211"
+		(property "Reference" "#PWR0221"
 			(at 91.44 54.61 0)
 			(effects
@@
 			(project ""
 				(path "/7eeba806-440e-4671-bc07-69fe183910a7/d2563b9c-21b7-43a8-ad57-d0568fac8495"
-					(reference "#PWR0211")
+					(reference "#PWR0221")
 					(unit 1)
 				)
