File: anamux.kicad_sch (KiCad schematic)
At the start: 4 parts, among them J52 Conn_01x08, U26 TMUX4051

Commit message: Update the design to a stackable one
Parts:
- removed D21: 1N5819WS, Diode_SMD:D_SOD-323, symbol Diode:1N5819WS
- J36: renamed from J52; value Conn_01x08 -> Conn_02x08_Pin; footprint HL_Connector_Pad_2.54mm:Pad_1x08_P2.54_1.7x1.7_Oct -> HL_Connector_Pad_2.54mm:Pad_2x09_P2.54_1.7x1.7_Rect-Oct; symbol Connector_Generic:Conn_01x08 -> Connector_Generic:Conn_02x09_Odd_Even; JLCPCB_CORRECTION 0;8.89;270 -> 1.27;-8.89;270; LCSC C492407 -> C5383108
- renumbered C55 to C65
Connections:
- net VDD is gone; now on net +12V: C65.1, U26.16 (VDD)
- net D: now also J36.2 (Pin_2)
- net GND: now also J36.1 (Pin_1), J36.11 (Pin_11), J36.13 (Pin_13), J36.15 (Pin_15), J36.17 (Pin_17), J36.3 (Pin_3), J36.5 (Pin_5), J36.7 (Pin_7), J36.9 (Pin_9)
- net S0: now also J36.4 (Pin_4); no longer J36.1 (Pin_1)
- net S1: now also J36.6 (Pin_6); no longer J36.2 (Pin_2)
- net S2: now also J36.8 (Pin_8); no longer J36.3 (Pin_3)
- net S3: now also J36.10 (Pin_10); no longer J36.4 (Pin_4)
- net S4: now also J36.12 (Pin_12); no longer J36.5 (Pin_5)
- net S5: now also J36.14 (Pin_14); no longer J36.6 (Pin_6)
- net S6: now also J36.16 (Pin_16); no longer J36.7 (Pin_7)
- net S7: now also J36.18 (Pin_18); no longer J36.8 (Pin_8)

Commit message: Fix some part numbers
Parts:
- J36: JLCPCB_CORRECTION 1.27;-8.89;270 -> 1.27;-10.16;270; LCSC C5383108 -> C492426
Changed lines of the file:
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@@
 			)
 		)
-		(property "LCSC" "C5383108"
+		(property "LCSC" "C492426"
 			(at 123.19 78.74 0)
 			(effects
@@
 			)
 		)
-		(property "JLCPCB_CORRECTION" "1.27;-8.89;270"
+		(property "JLCPCB_CORRECTION" "1.27;-10.16;270"
 			(at 123.19 78.74 0)
 			(effects
